File: eagle/RS232_SelfPowered_Opto.sch (EAGLE design)
At the start: 12 parts, among them IC1 ACPL-827, J2 PIC-UART-4P, J3 COMPORT-6PIN-NEW

Commit message: ...
Parts:
- IC1: value ACPL-827 -> PC827
Changed lines of the file:
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@@
 <setting verticaltext="up"/>
 </settings>
-<grid distance="0.1" unitdist="inch" unit="inch" style="lines" multiple="1" display="no" altdistance="0.01" altunitdist="inch" altunit="inch"/>
+<grid distance="0.05" unitdist="inch" unit="inch" style="lines" multiple="2" display="yes" altdistance="0.025" altunitdist="inch" altunit="inch"/>
 <layers>
 <layer number="1" name="Top" color="4" fill="1" visible="no" active="no"/>
@@
 <part name="C1" library="rcl" deviceset="CPOL-EU" device="E2.5-5" value="47u"/>
 <part name="D1" library="d" deviceset="1N4148" device="34-7V" value="1N914"/>
-<part name="IC1" library="opto-c" deviceset="ACPL-827" device=""/>
+<part name="IC1" library="opto-c" deviceset="ACPL-827" device="" value="PC827"/>
 <part name="R3" library="r" deviceset="R" device="0202/10-V" value="470"/>
 <part name="P+1" library="supply1" deviceset="+5V" device=""/>
