File: eagle/JDM2_2-Voltage_JmpConf+RxD.brd (EAGLE design)
At the start: 35.6 x 27.9 mm, 23 parts, among them J1 COM, J2 PIC-ICSP-ICSP, SW1 SL-SW-1P-2T-JPSW, T1 BC547, T2 BC547, T3 BC557

Commit message: ...
Routing:
- added copper zone on layer 16, net GND
Other:
- board outline removed
