File: eagle/JDM2_2-Voltage_JmpConf_6Pin_New.brd (EAGLE design)
At the start: 35.6 x 20.3 mm, 18 parts, among them J1 COMPORT-6PIN-NEW-L, J2 PIC-ICSP-ICSP, SW1 SL-SW-1P-2T-JPSW, T1 BC547, T2 BC547

Commit message: ...
Routing:
- added copper zone on layer 16, net GND
Other:
- board outline removed
