File: eagle/PIC32_JTAG.brd (EAGLE design)
At the start: 100 x 80 mm, 2 parts, among them IC1 PIC32MX460F512L

Commit message: ...
Other:
- board outline removed
Changed lines of the file:
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@@
 <board>
 <plain>
-<wire x1="0" y1="-1.38490625" x2="100" y2="-1.38490625" width="0" layer="20"/>
-<wire x1="100" y1="-1.38490625" x2="100" y2="78.61509375" width="0" layer="20"/>
-<wire x1="100" y1="78.61509375" x2="0" y2="78.61509375" width="0" layer="20"/>
-<wire x1="0" y1="78.61509375" x2="0" y2="-1.38490625" width="0" layer="20"/>
+<wire x1="0" y1="-1.38490625" x2="100" y2="-1.38490625" width="0" layer="47"/>
+<wire x1="100" y1="-1.38490625" x2="100" y2="78.61509375" width="0" layer="47"/>
+<wire x1="100" y1="78.61509375" x2="0" y2="78.61509375" width="0" layer="47"/>
+<wire x1="0" y1="78.61509375" x2="0" y2="-1.38490625" width="0" layer="47"/>
 <wire x1="3.352340625" y1="1.722953125" x2="15.922" y2="1.722953125" width="0.001" layer="51"/>
 <wire x1="15.922" y1="1.722953125" x2="18.43591875" y2="1.722953125" width="0.001" layer="51"/>
@@
 <contactref element="IC1" pad="13"/>
 <contactref element="U$1" pad="6"/>
-<wire x1="5.08" y1="21.47509375" x2="1.27" y2="21.47509375" width="0.254" layer="16"/>
-<wire x1="1.27" y1="21.47509375" x2="1.27" y2="-0.11490625" width="0.254" layer="16"/>
-<wire x1="1.27" y1="-0.11490625" x2="10.16" y2="-0.11490625" width="0.254" layer="16"/>
+<wire x1="5.08" y1="21.47509375" x2="1.27" y2="21.47509375" width="1.27" layer="16"/>
+<wire x1="1.27" y1="21.47509375" x2="1.27" y2="-0.11490625" width="1.27" layer="16"/>
+<wire x1="1.27" y1="-0.11490625" x2="10.16" y2="-0.11490625" width="1.27" layer="16"/>
 <wire x1="10.16" y1="-0.11490625" x2="10.16" y2="1.02509375" width="0" layer="19" extent="1-16"/>
 </signal>
