File: eagle/PIC18F2550-USB+ICSP-Board.sch (EAGLE design)
At the start: 17 parts, among them J1 PIC-ICSP-ICSP, J2 USB-PRINT, J3 RA[0..4], J4 RC[0..3], J5 PWR+SCI+USB, J6 RB[0..7], Q1 20MHz

Commit message: ...
Parts:
- LED1: device led:LED3MM -> led:LED5MM
- R1: device r:R0202/10 -> r:R0204/10
- R2, R3: device r:R0202/7-V -> r:R0204/7-V
Changed lines of the file:
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@@
 <part name="U$3" library="pad" deviceset="GND" device=""/>
 <part name="U$5" library="pad" deviceset="GND" device=""/>
-<part name="R1" library="r" deviceset="R" device="0202/10" value="330"/>
-<part name="LED1" library="led" deviceset="LED" device="3MM"/>
+<part name="R1" library="r" deviceset="R" device="0204/10" value="330"/>
+<part name="LED1" library="led" deviceset="LED" device="5MM"/>
 <part name="VDD1" library="supply1" deviceset="VDD" device=""/>
 <part name="VDD2" library="supply1" deviceset="VDD" device=""/>
@@
 <part name="J6" library="pinconn" deviceset="CONN-8P" device="" value="RB[0..7]"/>
 <part name="J3" library="pinconn" deviceset="CONN-5P" device="" value="RA[0..4]"/>
-<part name="R2" library="r" deviceset="R" device="0202/7-V" value="100"/>
-<part name="R3" library="r" deviceset="R" device="0202/7-V" value="100"/>
+<part name="R2" library="r" deviceset="R" device="0204/7-V" value="100"/>
+<part name="R3" library="r" deviceset="R" device="0204/7-V" value="100"/>
 <part name="U$1" library="mcu" deviceset="PIC18F2550-I/SP" device="-V" value="PIC18F2550-I/SP-V"/>
 </parts>

Commit message: ...
Parts:
- U$1: value PIC18F2550-I/SP-V -> PIC18F2550-I/SPLABEL; device mcu:PIC18F2550-I/SP-V -> mcu:PIC18F2550-I/SPLABEL
Connections:
- new net VCC: C2.1, C5.+, J2.VBUS, J5.6, R1.2, U$1.VDD
- net N$20: now also LED1.C; no longer J3.5
- net N$5: now also J3.5; no longer LED1.C
- net VDD: no longer C2.1, C5.+, J2.VBUS, J5.6, R1.2, U$1.VDD
Other:
- moved on the sheet: J5, J6, LED1, R1
