File: eagle/MHBP-LCD-Adapter.brd (EAGLE design)
At the start: 40.6 x 27.9 mm, 4 parts, among them J1 HD44780-4BITLCD44780-8P

Commit message: ...
Parts:
- moved R2 0.63 mm to (38.1, 24.1)
Routing:
- net N$4: track 3.18 -> 3.81 mm
