File: eagle/7seg-2.54.sch (EAGLE design)
At the start: 14 parts, among them J1 CONN-8P, J2 CONN-4P-4P

Commit message: ...
Parts:
- R1, R2, R3, R4, R5, R6, R7, R8: value (none) -> 330
Connections:
- net C1: no longer U$1.C@2
- net C2: no longer U$2.C@2
- net C3: no longer U$3.C@2
- net C4: no longer U$4.C@2

Commit message: ...
Other:
- moved on the sheet: R1, R2, R3, R4, R5, R6, R7, R8
Changed lines of the file:
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@@
 <setting verticaltext="up"/>
 </settings>
-<grid distance="0.1" unitdist="inch" unit="inch" style="lines" multiple="1" display="yes" altdistance="2" altunitdist="inch" altunit="inch"/>
+<grid distance="0.05" unitdist="inch" unit="inch" style="lines" multiple="2" display="yes" altdistance="4" altunitdist="inch" altunit="inch"/>
 <layers>
 <layer number="1" name="Top" color="4" fill="1" visible="no" active="no"/>
@@
 <instance part="U$3" gate="G$1" x="81.28" y="25.4"/>
 <instance part="U$4" gate="G$1" x="111.76" y="25.4"/>
-<instance part="R1" gate="1" x="55.88" y="-30.48"/>
-<instance part="R2" gate="1" x="60.96" y="-30.48"/>
-<instance part="R3" gate="1" x="66.04" y="-30.48"/>
-<instance part="R4" gate="1" x="71.12" y="-30.48"/>
-<instance part="R5" gate="1" x="76.2" y="-30.48"/>
-<instance part="R6" gate="1" x="81.28" y="-30.48"/>
-<instance part="R7" gate="1" x="86.36" y="-30.48"/>
-<instance part="R8" gate="1" x="91.44" y="-30.48"/>
+<instance part="R1" gate="1" x="81.28" y="-30.48" rot="R90"/>
+<instance part="R2" gate="1" x="76.2" y="-30.48" rot="R90"/>
+<instance part="R3" gate="1" x="86.36" y="-30.48" rot="R90"/>
+<instance part="R4" gate="1" x="60.96" y="-30.48" rot="R90"/>
+<instance part="R5" gate="1" x="55.88" y="-30.48" rot="R90"/>
+<instance part="R6" gate="1" x="71.12" y="-30.48" rot="R90"/>
+<instance part="R7" gate="1" x="66.04" y="-30.48" rot="R90"/>
+<instance part="R8" gate="1" x="91.44" y="-30.48" rot="R90"/>
 <instance part="J1" gate="G$1" x="113.03" y="-52.07" rot="MR180"/>
 <instance part="J2" gate="G$1" x="116.84" y="-22.86"/>
@@
 <segment>
 <wire x1="88.9" y1="-15.24" x2="91.44" y2="-17.78" width="0.1524" layer="91"/>
-<wire x1="91.44" y1="-17.78" x2="96.52" y2="-30.48" width="0.1524" layer="91"/>
+<wire x1="91.44" y1="-17.78" x2="91.44" y2="-25.4" width="0.1524" layer="91"/>
 <pinref part="R8" gate="1" pin="2"/>
 <label x="88.9" y="-22.86" size="1.778" layer="95"/>
@@
 </segment>
 <segment>
-<wire x1="53.34" y1="-15.24" x2="55.88" y2="-17.78" width="0.1524" layer="91"/>
-<wire x1="55.88" y1="-17.78" x2="60.96" y2="-30.48" width="0.1524" layer="91"/>
+<wire x1="78.74" y1="-15.24" x2="81.28" y2="-17.78" width="0.1524" layer="91"/>
+<wire x1="81.28" y1="-17.78" x2="81.28" y2="-25.4" width="0.1524" layer="91"/>
 <pinref part="R1" gate="1" pin="2"/>
-<label x="54.61" y="-22.86" size="1.778" layer="95"/>
+<label x="78.74" y="-22.86" size="1.778" layer="95"/>
 </segment>
 </net>
@@
 </segment>
 <segment>
-<wire x1="58.42" y1="-15.24" x2="60.96" y2="-17.78" width="0.1524" layer="91"/>
-<wire x1="60.96" y1="-17.78" x2="66.04" y2="-30.48" width="0.1524" layer="91"/>
+<wire x1="73.66" y1="-15.24" x2="76.2" y2="-17.78" width="0.1524" layer="91"/>
+<wire x1="76.2" y1="-17.78" x2="76.2" y2="-25.4" width="0.1524" layer="91"/>
 <pinref part="R2" gate="1" pin="2"/>
-<label x="59.69" y="-22.86" size="1.778" layer="95"/>
+<label x="73.66" y="-22.86" size="1.778" layer="95"/>
 </segment>
 </net>
@@
 </segment>
 <segment>
-<wire x1="63.5" y1="-15.24" x2="66.04" y2="-17.78" width="0.1524" layer="91"/>
-<wire x1="66.04" y1="-17.78" x2="71.12" y2="-30.48" width="0.1524" layer="91"/>
+<wire x1="83.82" y1="-15.24" x2="86.36" y2="-17.78" width="0.1524" layer="91"/>
+<wire x1="86.36" y1="-17.78" x2="86.36" y2="-25.4" width="0.1524" layer="91"/>
 <pinref part="R3" gate="1" pin="2"/>
-<label x="64.77" y="-21.59" size="1.778" layer="95"/>
+<label x="83.82" y="-22.86" size="1.778" layer="95"/>
 </segment>
 </net>
@@
 </segment>
 <segment>
-<wire x1="68.58" y1="-15.24" x2="71.12" y2="-17.78" width="0.1524" layer="91"/>
-<wire x1="71.12" y1="-17.78" x2="76.2" y2="-30.48" width="0.1524" layer="91"/>
+<wire x1="58.42" y1="-15.24" x2="60.96" y2="-17.78" width="0.1524" layer="91"/>
+<wire x1="60.96" y1="-17.78" x2="60.96" y2="-25.4" width="0.1524" layer="91"/>
 <pinref part="R4" gate="1" pin="2"/>
-<label x="68.58" y="-22.86" size="1.778" layer="95"/>
+<label x="58.42" y="-22.86" size="1.778" layer="95"/>
 </segment>
 </net>
@@
 </segment>
 <segment>
-<wire x1="73.66" y1="-15.24" x2="76.2" y2="-17.78" width="0.1524" layer="91"/>
-<wire x1="76.2" y1="-17.78" x2="81.28" y2="-30.48" width="0.1524" layer="91"/>
+<wire x1="53.34" y1="-15.24" x2="55.88" y2="-17.78" width="0.1524" layer="91"/>
+<wire x1="55.88" y1="-17.78" x2="55.88" y2="-25.4" width="0.1524" layer="91"/>
 <pinref part="R5" gate="1" pin="2"/>
-<label x="73.66" y="-22.86" size="1.778" layer="95"/>
+<label x="53.34" y="-22.86" size="1.778" layer="95"/>
 </segment>
 </net>
@@
 </segment>
 <segment>
-<wire x1="78.74" y1="-15.24" x2="81.28" y2="-17.78" width="0.1524" layer="91"/>
-<wire x1="81.28" y1="-17.78" x2="86.36" y2="-30.48" width="0.1524" layer="91"/>
+<wire x1="68.58" y1="-15.24" x2="71.12" y2="-17.78" width="0.1524" layer="91"/>
+<wire x1="71.12" y1="-17.78" x2="71.12" y2="-25.4" width="0.1524" layer="91"/>
 <pinref part="R6" gate="1" pin="2"/>
-<label x="78.74" y="-22.86" size="1.778" layer="95"/>
+<label x="68.58" y="-22.86" size="1.778" layer="95"/>
 </segment>
 </net>
@@
 </segment>
 <segment>
-<wire x1="83.82" y1="-15.24" x2="86.36" y2="-17.78" width="0.1524" layer="91"/>
-<wire x1="86.36" y1="-17.78" x2="91.44" y2="-30.48" width="0.1524" layer="91"/>
+<wire x1="63.5" y1="-15.24" x2="66.04" y2="-17.78" width="0.1524" layer="91"/>
+<wire x1="66.04" y1="-17.78" x2="66.04" y2="-25.4" width="0.1524" layer="91"/>
 <pinref part="R7" gate="1" pin="2"/>
-<label x="83.82" y="-22.86" size="1.778" layer="95"/>
+<label x="63.5" y="-22.86" size="1.778" layer="95"/>
 </segment>
 </net>
@@
 <segment>
 <pinref part="R1" gate="1" pin="1"/>
-<wire x1="50.8" y1="-30.48" x2="55.88" y2="-48.26" width="0.1524" layer="91"/>
+<wire x1="81.28" y1="-35.56" x2="81.28" y2="-48.26" width="0.1524" layer="91"/>
 <pinref part="J1" gate="G$1" pin="3"/>
-<wire x1="55.88" y1="-48.26" x2="111.76" y2="-48.26" width="0.1524" layer="91"/>
+<wire x1="81.28" y1="-48.26" x2="111.76" y2="-48.26" width="0.1524" layer="91"/>
 <label x="101.6" y="-48.26" size="1.778" layer="95"/>
 </segment>
@@
 <segment>
 <pinref part="R2" gate="1" pin="1"/>
-<wire x1="55.88" y1="-30.48" x2="60.96" y2="-50.8" width="0.1524" layer="91"/>
-<wire x1="60.96" y1="-50.8" x2="111.76" y2="-50.8" width="0.1524" layer="91"/>
+<wire x1="76.2" y1="-35.56" x2="76.2" y2="-50.8" width="0.1524" layer="91"/>
+<wire x1="76.2" y1="-50.8" x2="111.76" y2="-50.8" width="0.1524" layer="91"/>
 <pinref part="J1" gate="G$1" pin="4"/>
 <label x="101.6" y="-50.8" size="1.778" layer="95"/>
@@
 <segment>
 <pinref part="R3" gate="1" pin="1"/>
-<wire x1="60.96" y1="-30.48" x2="66.04" y2="-45.72" width="0.1524" layer="91"/>
-<wire x1="66.04" y1="-45.72" x2="111.76" y2="-45.72" width="0.1524" layer="91"/>
+<wire x1="86.36" y1="-35.56" x2="86.36" y2="-45.72" width="0.1524" layer="91"/>
+<wire x1="86.36" y1="-45.72" x2="111.76" y2="-45.72" width="0.1524" layer="91"/>
 <pinref part="J1" gate="G$1" pin="2"/>
 <label x="101.6" y="-45.72" size="1.778" layer="95"/>
@@
 <segment>
 <pinref part="R4" gate="1" pin="1"/>
-<wire x1="66.04" y1="-30.48" x2="71.12" y2="-58.42" width="0.1524" layer="91"/>
-<wire x1="71.12" y1="-58.42" x2="111.76" y2="-58.42" width="0.1524" layer="91"/>
+<wire x1="60.96" y1="-35.56" x2="60.96" y2="-58.42" width="0.1524" layer="91"/>
+<wire x1="60.96" y1="-58.42" x2="111.76" y2="-58.42" width="0.1524" layer="91"/>
 <pinref part="J1" gate="G$1" pin="7"/>
 <label x="101.6" y="-58.42" size="1.778" layer="95"/>
@@
 <segment>
 <pinref part="R5" gate="1" pin="1"/>
-<wire x1="71.12" y1="-30.48" x2="76.2" y2="-60.96" width="0.1524" layer="91"/>
+<wire x1="55.88" y1="-35.56" x2="55.88" y2="-60.96" width="0.1524" layer="91"/>
 <pinref part="J1" gate="G$1" pin="8"/>
-<wire x1="76.2" y1="-60.96" x2="111.76" y2="-60.96" width="0.1524" layer="91"/>
+<wire x1="55.88" y1="-60.96" x2="111.76" y2="-60.96" width="0.1524" layer="91"/>
 <label x="101.6" y="-60.96" size="1.778" layer="95"/>
 </segment>
@@
 <segment>
 <pinref part="R6" gate="1" pin="1"/>
-<wire x1="76.2" y1="-30.48" x2="81.28" y2="-53.34" width="0.1524" layer="91"/>
+<wire x1="71.12" y1="-35.56" x2="71.12" y2="-53.34" width="0.1524" layer="91"/>
 <pinref part="J1" gate="G$1" pin="5"/>
-<wire x1="81.28" y1="-53.34" x2="111.76" y2="-53.34" width="0.1524" layer="91"/>
+<wire x1="71.12" y1="-53.34" x2="111.76" y2="-53.34" width="0.1524" layer="91"/>
 <label x="101.6" y="-53.34" size="1.778" layer="95"/>
 </segment>
@@
 <pinref part="R7" gate="1" pin="1"/>
 <pinref part="J1" gate="G$1" pin="6"/>
-<wire x1="81.28" y1="-30.48" x2="86.36" y2="-55.88" width="0.1524" layer="91"/>
-<wire x1="86.36" y1="-55.88" x2="111.76" y2="-55.88" width="0.1524" layer="91"/>
+<wire x1="66.04" y1="-35.56" x2="66.04" y2="-55.88" width="0.1524" layer="91"/>
+<wire x1="66.04" y1="-55.88" x2="111.76" y2="-55.88" width="0.1524" layer="91"/>
 <label x="101.6" y="-55.88" size="1.778" layer="95"/>
 </segment>
@@
 <segment>
 <pinref part="R8" gate="1" pin="1"/>
-<wire x1="86.36" y1="-30.48" x2="91.44" y2="-43.18" width="0.1524" layer="91"/>
+<wire x1="91.44" y1="-35.56" x2="91.44" y2="-43.18" width="0.1524" layer="91"/>
 <wire x1="91.44" y1="-43.18" x2="111.76" y2="-43.18" width="0.1524" layer="91"/>
 <pinref part="J1" gate="G$1" pin="1"/>
