File: eagle/7seg-2.54-new.brd (EAGLE design)
At the start: 25 parts, among them J1 CONN-8P, J2 CONN-4P-4P, J3 CONN-6P, SW1 PB-1P-1T2P1T-2X3, SW2 PB-1P-1T2P1T-2X3, SW3 PB-1P-1T2P1T-2X3, SW4 PB-1P-1T2P1T-2X3

Commit message: ...
Parts:
- R9: value 10k -> 10kΩ
Changed lines of the file:
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@@
 <element name="D1" library="d" package="DO34-2,5" value="" x="6.35" y="25.4"/>
 <element name="VCC" library="pad" package="SPAD" value="SPAD" x="17.78" y="2.54"/>
-<element name="R9" library="r" package="0202/5-V" value="10k" x="12.7" y="2.54" rot="R270"/>
+<element name="R9" library="r" package="0202/5-V" value="10kΩ" x="12.7" y="2.54" rot="R270"/>
 </elements>
 <signals>
