File: eagle/7seg.sch (EAGLE design)
At the start: 14 parts, among them J1 CONN-8P, J2 CONN-4P-4P

Commit message: ...
Parts:
- R1, R2, R3, R4, R5, R6, R7, R8: value 330Ω -> (none); device r:R0202/5-V -> r:R0202/7-V
- U$1, U$2, U$3, U$4: value TDSO1160-2.54 -> TDSO1160; device lcd:TDSO1160-2.54 -> lcd:TDSO1160
Connections:
- net DP renamed P
- net _A renamed N$1
- net _B renamed N$2
- net _C renamed N$3
- net _D renamed N$4
- net _DP renamed N$8
- net _E renamed N$5
- net _F renamed N$6
- net _G renamed N$7
