File: eagle/JDM2_2-Voltage.sch (EAGLE design)
At the start: 19 parts, among them J1 COMPORT-6PIN, J2 PIC-ICSPICSP, SW1 SL-SW-2P-2T-S, T1 BC547CBE-A, T2 BC547CBE

Commit message: ...
Parts:
- C1: value 100uF -> 100μF
- C2: value 22uF -> 22μF
- R1: value 10k -> 10kΩ
- R2: value 1.5k -> 1.5kΩ
- R3: value 100 -> 100Ω
Changed lines of the file:
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@@
 <part name="D6" library="d" deviceset="1N4148" device="34-7" value="1N4148"/>
 <part name="D7" library="d" deviceset="1N4148" device="34-7" value="1N4148"/>
-<part name="R2" library="r" deviceset="R" device="0202/7" value="1.5k"/>
-<part name="R1" library="r" deviceset="R" device="0202/7" value="10k"/>
+<part name="R2" library="r" deviceset="R" device="0202/7" value="1.5kΩ"/>
+<part name="R1" library="r" deviceset="R" device="0202/7" value="10kΩ"/>
 <part name="T1" library="t" deviceset="BC547" device="CBE-A" value="BC547CBE-A"/>
 <part name="T2" library="t" deviceset="BC547" device="CBE" value="BC547CBE"/>
-<part name="C1" library="c" deviceset="CPOL" device="E5-4" value="100uF"/>
-<part name="C2" library="c" deviceset="CPOL" device="E2,5-4" value="22uF"/>
+<part name="C1" library="c" deviceset="CPOL" device="E5-4" value="100μF"/>
+<part name="C2" library="c" deviceset="CPOL" device="E2,5-4" value="22μF"/>
 <part name="VSS" library="supply1" deviceset="GND" device="" value="VSS"/>
 <part name="VSS1" library="supply1" deviceset="GND" device="" value="VSS"/>
@@
 <part name="SUPPLY1" library="supply2" deviceset="VPP" device=""/>
 <part name="D3" library="led" deviceset="LED" device="3MM" value="Vpp"/>
-<part name="R3" library="r" deviceset="R" device="0202/5" value="100"/>
+<part name="R3" library="r" deviceset="R" device="0202/5" value="100Ω"/>
 <part name="J1" library="pinconn" deviceset="COMPORT-6PIN" device=""/>
 <part name="J2" library="pinconn" deviceset="PIC-ICSP" device="ICSP" value="PIC-ICSPICSP"/>
