File: eagle/JDM2_2-Voltage_JmpConf_6Pin_New.sch (EAGLE design)
At the start: 18 parts, among them J1 COMPORT-6PIN-NEW-L, J2 PIC-ICSP-ICSP, SW1 SL-SW-1P-2T-JPSW, T1 BC547, T2 BC547

Commit message: ...
Parts:
- C1: value 100uF -> 100μF
- C2: value 22uF -> 22μF
- R1: value 10k -> 10kΩ
- R2: value 1.5k -> 1.5kΩ
- R3: value 100 -> 100Ω
Changed lines of the file:
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@@
 <part name="D6" library="d" deviceset="1N4148" device="34-5V" value="1N4148"/>
 <part name="D7" library="d" deviceset="1N4148" device="34-7V" value="1N4148"/>
-<part name="R2" library="r" deviceset="R" device="0202/7-V" value="1.5k"/>
-<part name="R1" library="r" deviceset="R" device="0202/7-V" value="10k"/>
+<part name="R2" library="r" deviceset="R" device="0202/7-V" value="1.5kΩ"/>
+<part name="R1" library="r" deviceset="R" device="0202/7-V" value="10kΩ"/>
 <part name="T1" library="t" deviceset="BC547" device="CBE" value="BC547"/>
 <part name="T2" library="t" deviceset="BC547" device="CBE" value="BC547"/>
-<part name="C1" library="c" deviceset="CPOL" device="E2,5-5/V" value="100uF"/>
-<part name="C2" library="c" deviceset="CPOL" device="E2,5-4/V" value="22uF"/>
+<part name="C1" library="c" deviceset="CPOL" device="E2,5-5/V" value="100μF"/>
+<part name="C2" library="c" deviceset="CPOL" device="E2,5-4/V" value="22μF"/>
 <part name="D6B" library="d" deviceset="Z-DIODE" device="34Z7V" value="Z=5.1V"/>
 <part name="SUPPLY1" library="supply2" deviceset="VPP" device=""/>
-<part name="R3" library="r" deviceset="R" device="0202/7" value="100"/>
+<part name="R3" library="r" deviceset="R" device="0202/7" value="100Ω"/>
 <part name="J2" library="pinconn" deviceset="PIC-ICSP" device="-ICSP" value="PIC-ICSP-ICSP"/>
 <part name="SUPPLY2" library="supply2" deviceset="VPP" device=""/>
