File: eagle/JDM2_2-Voltage_SW1P.brd (EAGLE design)
At the start: 20 parts, among them J1 COMPORT-6PIN, J2 PIC-ICSPICSP, SW1 SL-SW-1P-2T-H, T1 BC547, T2 BC547

Commit message: ...
Parts:
- C1: value 100uF -> 100μF
- C2: value 22uF -> 22μF
- R1: value 10k -> 10kΩ
- R2: value 1.5k -> 1.5kΩ
- R3: value 100 -> 100Ω
Changed lines of the file:
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@@
 </autorouter>
 <elements>
-<element name="C1" library="c" package="E2,5-5" value="100uF" x="21.59" y="15.24" smashed="yes" rot="R90">
+<element name="C1" library="c" package="E2,5-5" value="100μF" x="21.59" y="15.24" smashed="yes" rot="R90">
 <attribute name="NAME" x="17.907" y="15.24" size="1.016" layer="25" rot="R180" align="center-right"/>
 <attribute name="VALUE" x="24.384" y="15.24" size="0.4064" layer="27" align="center-left"/>
 </element>
-<element name="C2" library="c" package="E2,5-4" value="22uF" x="24.13" y="10.16" smashed="yes">
+<element name="C2" library="c" package="E2,5-4" value="22μF" x="24.13" y="10.16" smashed="yes">
 <attribute name="NAME" x="21.59" y="10.16" size="0.8128" layer="25" align="center-right"/>
 <attribute name="VALUE" x="26.416" y="10.16" size="0.4064" layer="27" align="center-left"/>
@@
 <attribute name="NAME" x="-0.254" y="0" size="1.016" layer="25" rot="R180" align="top-left"/>
 </element>
-<element name="R1" library="r" package="0202/7-V" value="10k" x="8.89" y="7.62"/>
-<element name="R2" library="r" package="0202/7-V" value="1.5k" x="6.35" y="7.62"/>
+<element name="R1" library="r" package="0202/7-V" value="10kΩ" x="8.89" y="7.62"/>
+<element name="R2" library="r" package="0202/7-V" value="1.5kΩ" x="6.35" y="7.62"/>
 <element name="T1" library="t" package="TO92-CBE" value="BC547" x="6.35" y="16.51" smashed="yes">
 <attribute name="NAME" x="7.62" y="17.78" size="0.6096" layer="25" ratio="10" align="center"/>
@@
 <attribute name="VALUE" x="10.16" y="2.4765" size="0.4064" layer="27" ratio="10" rot="R180" align="center"/>
 </element>
-<element name="R3" library="r" package="0202/10" value="100" x="19.05" y="1.27" rot="R90"/>
+<element name="R3" library="r" package="0202/10" value="100Ω" x="19.05" y="1.27" rot="R90"/>
 <element name="J2" library="pinconn" package="PIC-ICSP" value="PIC-ICSPICSP" x="36.83" y="11.43" smashed="yes" rot="R270">
 <attribute name="NAME" x="35.052" y="5.588" size="0.8128" layer="25" rot="R270" align="top-left"/>
