File: eagle/JDM2_Low_Voltage.sch (EAGLE design)
At the start: 27 parts, among them J1 DUMMY, T1 BC547, T2 BC547, T3 2N7000

Commit message: ...
Parts:
- C1: value 100uF -> 100μF
- C2: value 22uF -> 22μF
- R1: value 10k -> 10kΩ
- R2: value 1.5k -> 1.5kΩ
- R4: value 1K -> 1kΩ
- R5: value 15K -> 15kΩ
- R6: value 4.7k -> 4.7kΩ
- R7: value 1k -> 1kΩ
Changed lines of the file:
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@@
 <part name="D4" library="JDM2" deviceset="1N4148" device="-2.54" value="1N4148"/>
 <part name="D5" library="JDM2" deviceset="1N4148" device="-18" value="1N4148"/>
-<part name="R6" library="JDM2" deviceset="RES" device="-0204-7" value="4.7k"/>
-<part name="R7" library="JDM2" deviceset="RES" device="-0204-7" value="1k"/>
-<part name="R2" library="JDM2" deviceset="RES" device="-0204-7" value="1.5k"/>
-<part name="R1" library="JDM2" deviceset="RES" device="-0207-10" value="10k"/>
+<part name="R6" library="JDM2" deviceset="RES" device="-0204-7" value="4.7kΩ"/>
+<part name="R7" library="JDM2" deviceset="RES" device="-0204-7" value="1kΩ"/>
+<part name="R2" library="JDM2" deviceset="RES" device="-0204-7" value="1.5kΩ"/>
+<part name="R1" library="JDM2" deviceset="RES" device="-0207-10" value="10kΩ"/>
 <part name="T1" library="JDM2" deviceset="BC547" device="" value="BC547"/>
 <part name="T2" library="JDM2" deviceset="BC547" device="" value="BC547"/>
-<part name="C1" library="rcl" deviceset="CPOL-EU" device="E2.5-5" value="100uF"/>
-<part name="C2" library="rcl" deviceset="CPOL-EU" device="E2.5-5" value="22uF"/>
+<part name="C1" library="rcl" deviceset="CPOL-EU" device="E2.5-5" value="100μF"/>
+<part name="C2" library="rcl" deviceset="CPOL-EU" device="E2.5-5" value="22μF"/>
 <part name="LED2" library="1dmf" deviceset="LED" device="" value="Vpp"/>
 <part name="LED1" library="1dmf" deviceset="LED" device="" value="Power"/>
@@
 <part name="VSS" library="supply1" deviceset="GND" device="" value="VSS"/>
 <part name="VSS1" library="supply1" deviceset="GND" device="" value="VSS"/>
-<part name="R4" library="JDM2" deviceset="RES" device="-0207-10" value="1K"/>
-<part name="R5" library="JDM2" deviceset="RES" device="-0207-10" value="15K"/>
+<part name="R4" library="JDM2" deviceset="RES" device="-0207-10" value="1kΩ" />
+<part name="R5" library="JDM2" deviceset="RES" device="-0207-10" value="15kΩ" />
 <part name="D7" library="JDM2" deviceset="1N4148" device="-2.54A" value="2N4148"/>
 <part name="V1" library="supply2" deviceset="GND" device="" value="VSS"/>
