File: eagle/PicKit2-v1.2.brd (EAGLE design)
At the start: 160 x 100 mm, 36 parts, among them IC1 PIC18F2550_28DIP, J1 USB-PRINT, Q1 20 MHz, Q2 2N3906, SW1 PB-1P-1T, T1 2N3904, T2 2N3904, T3 2N3904

Commit message: ...
Parts:
- L1: device l:L-09R -> l:L-8R
Changed lines of the file:
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@@
           <attribute name="OC_FARNELL" value="1523822" x="41.91" y="34.29" size="1.778" layer="27" rot="R270" display="off" />
         </element>
-        <element name="L1" library="l" package="L-09R" value="680 uH" x="55.88" y="12.7" rot="R90" />
+        <element name="L1" library="l" package="L-8R" value="680 uH" x="55.88" y="12.7" rot="R90" />
         <element name="LED1" library="d" package="LED_3MM" value="Red Busy" x="-60.96" y="52.07" />
         <element name="LED2" library="led" package="LED3MM" value="Green Power" x="-52.07" y="52.07" />

Commit message: ...
Parts:
- C3: value 47 uF -> 47 μF
- C4: value 0.47 uF -> 0.47 μF
- C5: value 0.1 uF -> 0.1 μF
- L1: value 680 uH -> 680μH
- R1, R6, R7, R9: value 4.7 K -> 4.7kΩ
- R10, R11, R5: value 10 K -> 10kΩ
- R12: value 100 K -> 100kΩ
- R13, R2, R3, R4: value 100 -> 100Ω
- R14: value 1 K -> 1kΩ
- R15, R16: value 330 -> 330Ω
- R17: value 22 K -> 22kΩ
- R8: value 2.7 K -> 2.7kΩ
Changed lines of the file:
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@@
         <element name="C1" library="c" package="C025-020X036" value="22p" x="19.05" y="48.26" rot="R180" />
         <element name="C2" library="c" package="C025-020X036" value="22p" x="7.62" y="35.56" rot="R90" />
-        <element name="C3" library="rcl" package="E2,5-6E" value="47 uF" x="33.02" y="12.7" rot="R270" />
-        <element name="C4" library="c" package="C050-030X075" value="0.47 uF" x="27.94" y="15.24" rot="R270" />
-        <element name="C5" library="c" package="C050-024X044" value="0.1 uF" x="60.96" y="17.78" />
+        <element name="C3" library="rcl" package="E2,5-6E" value="47 μF" x="33.02" y="12.7" rot="R270" />
+        <element name="C4" library="c" package="C050-030X075" value="0.47 μF" x="27.94" y="15.24" rot="R270" />
+        <element name="C5" library="c" package="C050-024X044" value="0.1 μF" x="60.96" y="17.78" />
         <element name="D2" library="d" package="DO34Z10" value="1N5817-B" x="55.88" y="26.67" rot="R90" />
         <element name="D3" library="d" package="DO34-10" value="" x="60.96" y="7.62" rot="R180" />
@@
           <attribute name="OC_FARNELL" value="1523822" x="41.91" y="34.29" size="1.778" layer="27" rot="R270" display="off" />
         </element>
-        <element name="L1" library="l" package="L-8R" value="680 uH" x="55.88" y="12.7" rot="R90" />
+        <element name="L1" library="l" package="L-8R" value="680μH" x="55.88" y="12.7" rot="R90" />
         <element name="LED1" library="d" package="LED_3MM" value="Red Busy" x="-60.96" y="52.07" />
         <element name="LED2" library="led" package="LED3MM" value="Green Power" x="-52.07" y="52.07" />
         <element name="Q1" library="special" package="QS" value="20 MHz" x="43.18" y="71.12" rot="R180" />
         <element name="Q2" library="t" package="TO92" value="2N3906" x="60.96" y="25.4" rot="R180" />
-        <element name="R1" library="r" package="0204/10" value="4.7 K" x="30.48" y="45.72" />
-        <element name="R10" library="r" package="0204/10" value="10 K" x="53.34" y="38.1" rot="R180" />
-        <element name="R11" library="r" package="0204/10" value="10 K" x="96.52" y="20.32" rot="R270" />
-        <element name="R12" library="r" package="0204/10" value="100 K" x="66.04" y="20.32" rot="R90" />
-        <element name="R13" library="r" package="0204/10" value="100" x="66.04" y="35.56" rot="R90" />
-        <element name="R14" library="r" package="0204/10" value="1 K" x="30.48" y="22.86" />
-        <element name="R15" library="r" package="0204/10" value="330" x="60.96" y="50.8" rot="R90" />
-        <element name="R16" library="r" package="0204/10" value="330" x="30.48" y="25.4" rot="R180" />
-        <element name="R17" library="r" package="0204/10" value="22 K" x="53.34" y="45.72" rot="R180" />
-        <element name="R2" library="r" package="0204/10" value="100" x="30.48" y="43.18" />
-        <element name="R3" library="r" package="0204/10" value="100" x="30.48" y="40.64" />
-        <element name="R4" library="r" package="0204/10" value="100" x="38.1" y="66.04" />
-        <element name="R5" library="r" package="0204/10" value="10 K" x="30.48" y="35.56" />
-        <element name="R6" library="r" package="0204/10" value="4.7 K" x="17.78" y="40.64" />
-        <element name="R7" library="r" package="0204/10" value="4.7 K" x="17.78" y="43.18" />
-        <element name="R8" library="r" package="0204/10" value="2.7 K" x="30.48" y="33.02" />
-        <element name="R9" library="r" package="0204/10" value="4.7 K" x="22.86" y="27.94" rot="R90" />
+        <element name="R1" library="r" package="0204/10" value="4.7kΩ" x="30.48" y="45.72" />
+        <element name="R10" library="r" package="0204/10" value="10kΩ" x="53.34" y="38.1" rot="R180" />
+        <element name="R11" library="r" package="0204/10" value="10kΩ" x="96.52" y="20.32" rot="R270" />
+        <element name="R12" library="r" package="0204/10" value="100kΩ" x="66.04" y="20.32" rot="R90" />
+        <element name="R13" library="r" package="0204/10" value="100Ω" x="66.04" y="35.56" rot="R90" />
+        <element name="R14" library="r" package="0204/10" value="1kΩ" x="30.48" y="22.86" />
+        <element name="R15" library="r" package="0204/10" value="330Ω" x="60.96" y="50.8" rot="R90" />
+        <element name="R16" library="r" package="0204/10" value="330Ω" x="30.48" y="25.4" rot="R180" />
+        <element name="R17" library="r" package="0204/10" value="22kΩ" x="53.34" y="45.72" rot="R180" />
+        <element name="R2" library="r" package="0204/10" value="100Ω" x="30.48" y="43.18" />
+        <element name="R3" library="r" package="0204/10" value="100Ω" x="30.48" y="40.64" />
+        <element name="R4" library="r" package="0204/10" value="100Ω" x="38.1" y="66.04" />
+        <element name="R5" library="r" package="0204/10" value="10kΩ" x="30.48" y="35.56" />
+        <element name="R6" library="r" package="0204/10" value="4.7kΩ" x="17.78" y="40.64" />
+        <element name="R7" library="r" package="0204/10" value="4.7kΩ" x="17.78" y="43.18" />
+        <element name="R8" library="r" package="0204/10" value="2.7kΩ" x="30.48" y="33.02" />
+        <element name="R9" library="r" package="0204/10" value="4.7kΩ" x="22.86" y="27.94" rot="R90" />
         <element name="SV1" library="con-lsta" package="FE06" value="" x="25.4" y="69.85" rot="R180">
           <attribute name="OC_NEWARK" value="unknown" x="25.4" y="69.85" size="1.778" layer="27" rot="R180" display="off" />
