File: eagle/PicKit2-v1.2.sch (EAGLE design)
At the start: 36 parts, among them IC1 PIC18F2550_28DIP, J1 USB-PRINT, Q1 20 MHz, Q2 2N3906, SW1 PB-1P-1T, T1 2N3904, T2 2N3904, T3 2N3904

Commit message: ...
Parts:
- C3: value 47 uF -> 47 μF
- C4: value 0.47 uF -> 0.47 μF
- C5: value 0.1 uF -> 0.1 μF
- L1: value 680 uH -> 680μH
- R13, R2, R3, R4: value 100 -> 100Ω
- R15, R16: value 330 -> 330Ω
Changed lines of the file:
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@@
 <part name="C2" library="c" deviceset="C" device="025-020X036" value="22p"/>
 <part name="R1" library="r" deviceset="R-H" device="0204/10" value="4.7 K"/>
-<part name="R2" library="r" deviceset="R-H" device="0204/10" value="100"/>
-<part name="R3" library="r" deviceset="R-H" device="0204/10" value="100"/>
-<part name="R4" library="r" deviceset="R-H" device="0204/10" value="100"/>
+<part name="R2" library="r" deviceset="R-H" device="0204/10" value="100Ω"/>
+<part name="R3" library="r" deviceset="R-H" device="0204/10" value="100Ω"/>
+<part name="R4" library="r" deviceset="R-H" device="0204/10" value="100Ω"/>
 <part name="R5" library="r" deviceset="R-H" device="0204/10" value="10 K"/>
 <part name="R6" library="r" deviceset="R-H" device="0204/10" value="4.7 K"/>
@@
 <part name="VDD1" library="supply1" deviceset="VDD" device=""/>
 <part name="D2" library="d" deviceset="Z-DIODE" device="34Z10" value="1N5817-B"/>
-<part name="L1" library="l" deviceset="L" device="-09R" value="680 uH"/>
+<part name="L1" library="l" deviceset="L" device="-09R" value="680μH"/>
 <part name="SV1" library="con-lsta" deviceset="FE06-1" device=""/>
 <part name="LED1" library="d" deviceset="LED" device="-3MM" value="Red Busy"/>
@@
 <part name="GND9" library="supply1" deviceset="GND" device=""/>
 <part name="R12" library="r" deviceset="R" device="0204/10" value="100 K"/>
-<part name="R13" library="r" deviceset="R" device="0204/10" value="100"/>
+<part name="R13" library="r" deviceset="R" device="0204/10" value="100Ω"/>
 <part name="GND10" library="supply1" deviceset="GND" device=""/>
-<part name="C3" library="rcl" deviceset="CPOL-EU" device="E2,5-6E" value="47 uF"/>
+<part name="C3" library="rcl" deviceset="CPOL-EU" device="E2,5-6E" value="47 μF"/>
 <part name="GND11" library="supply1" deviceset="GND" device=""/>
 <part name="R14" library="r" deviceset="R-H" device="0204/10" value="1 K"/>
 <part name="GND12" library="supply1" deviceset="GND" device=""/>
 <part name="VDD3" library="supply1" deviceset="VDD" device=""/>
-<part name="R15" library="r" deviceset="R" device="0204/10" value="330"/>
+<part name="R15" library="r" deviceset="R" device="0204/10" value="330Ω"/>
 <part name="GND13" library="supply1" deviceset="GND" device=""/>
-<part name="R16" library="r" deviceset="R" device="0204/10" value="330"/>
+<part name="R16" library="r" deviceset="R" device="0204/10" value="330Ω"/>
 <part name="GND14" library="supply1" deviceset="GND" device=""/>
-<part name="C4" library="c" deviceset="C" device="050-030X075" value="0.47 uF"/>
+<part name="C4" library="c" deviceset="C" device="050-030X075" value="0.47 μF"/>
 <part name="GND15" library="supply1" deviceset="GND" device=""/>
 <part name="GND16" library="supply1" deviceset="GND" device=""/>
@@
 <part name="VDD6" library="supply1" deviceset="VDD" device=""/>
 <part name="GND18" library="supply1" deviceset="GND" device=""/>
-<part name="C5" library="c" deviceset="C" device="050-024X044" value="0.1 uF"/>
+<part name="C5" library="c" deviceset="C" device="050-024X044" value="0.1 μF"/>
 <part name="D3" library="d" deviceset="DIODE" device="34-10"/>
 <part name="T1" library="t" deviceset="2N3904" device=""/>
