File: eagle/Pinguino-PIC18F2550-ICSP-Pk3.sch (EAGLE design)
At the start: 16 parts, among them IC1 PIC18F2550-I/SP-V, J1 USB-PRINT, J2 CONN-8P, J3 CONN-6P, J4 CONN-6P, J5 CONN-4P-4P, J7 PICKIT3-ICSP-PK3, Q1 20MHz, SW1 PB-1P-1T

Commit message: ...
Parts:
- C5: value 100uF -> 100μF
- R1: value 10k -> 10kΩ
Changed lines of the file:
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@@
 <part name="SW1" library="sw" deviceset="PB-1P-1T" device=""/>
 <part name="U$2" library="pad" deviceset="GND" device=""/>
-<part name="R1" library="r" deviceset="R" device="0204/10" value="10k"/>
+<part name="R1" library="r" deviceset="R" device="0204/10" value="10kΩ"/>
 <part name="Q1" library="q" deviceset="CRYSTAL" device="HC49" value="20MHz"/>
 <part name="C1" library="c" deviceset="C" device="025-015X024" value="15pF"/>
@@
 <part name="GND" library="pad" deviceset="GND" device=""/>
 <part name="C4" library="c" deviceset="C" device="025-015X024" value="100nF"/>
-<part name="C5" library="c" deviceset="CPOL" device="E2,5-4" value="100uF"/>
+<part name="C5" library="c" deviceset="CPOL" device="E2,5-4" value="100μF"/>
 <part name="U$1" library="pad" deviceset="VCC" device=""/>
 <part name="U$10" library="pad" deviceset="GND" device=""/>
