File: eagle/Pinguino-PIC18F2550.brd (EAGLE design)
At the start: 16 parts, among them IC1 PIC18F2550-I/SP-V, J1 USB-PRINT, J2 CONN-8P, J3 CONN-6P, J4 CONN-6P, J5 CONN-4P-4P, J6 PIC-ICSP, Q1 20MHz, SW1 PB-1P-1T

Commit message: ...
Parts:
- C5: value 100uF -> 100μF
- R1: value 10k -> 10kΩ
Changed lines of the file:
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@@
 <element name="C3" library="c" package="C075-032X103" value="220nF" x="12.7" y="19.05" rot="R270"/>
 <element name="C4" library="c" package="C025-015X024" value="100nF" x="30.48" y="34.29"/>
-<element name="C5" library="c" package="E2,5-4" value="100uF" x="35.56" y="33.02" rot="R90"/>
+<element name="C5" library="c" package="E2,5-4" value="100μF" x="35.56" y="33.02" rot="R90"/>
 <element name="IC1" library="mcu" package="DIL28-3/V" value="PIC18F2550-I/SP-V" x="21.59" y="39.37"/>
 <element name="J2" library="pinconn" package="CONN-8P" value="CONN-8P" x="40.64" y="38.1" rot="R90"/>
@@
 <element name="J5" library="pinconn" package="CONN-4P" value="CONN-4P-4P" x="2.54" y="26.67" rot="R270"/>
 <element name="Q1" library="q" package="HC49" value="20MHz" x="12.7" y="35.56" rot="R180"/>
-<element name="R1" library="r" package="0204/10" value="10k" x="17.78" y="58.42" rot="R180"/>
+<element name="R1" library="r" package="0204/10" value="10kΩ" x="17.78" y="58.42" rot="R180"/>
 <element name="SW1" library="sw" package="PB-1P1T" value="PB-1P-1T" x="7.62" y="60.96" rot="R180"/>
 <element name="J6" library="pinconn" package="CONN-5P" value="PIC-ICSP" x="20.32" y="66.04"/>
