File: eagle/RS232_2xNPN_FTDI_PowerSel.brd (EAGLE design)
At the start: 10 parts, among them J1 FTDI232-BO-5P-L, J2 PIC-UART-X, SW1 SL-SW-1P-2T-JPSW, T1 BC547, T2 BC547

Commit message: ...
Parts:
- R1: value 4.7k -> 4.7kΩ
- R4: value 10k -> 10kΩ
- R5, R6: value 1k -> 1kΩ
Changed lines of the file:
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@@
 <elements>
 <element name="D1" library="d" package="DO34-5V" value="1N4148" x="17.78" y="7.62" rot="R180"/>
-<element name="R1" library="r" package="0202/7" value="4.7k" x="11.43" y="7.62" rot="R180"/>
-<element name="R4" library="r" package="0202/7" value="10k" x="19.05" y="12.7" rot="R180"/>
-<element name="R5" library="r" package="0202/7-V" value="1k" x="20.32" y="6.35" rot="R180"/>
+<element name="R1" library="r" package="0202/7" value="4.7kΩ" x="11.43" y="7.62" rot="R180"/>
+<element name="R4" library="r" package="0202/7" value="10kΩ" x="19.05" y="12.7" rot="R180"/>
+<element name="R5" library="r" package="0202/7-V" value="1kΩ" x="20.32" y="6.35" rot="R180"/>
 <element name="T1" library="t" package="TO92-CBE" value="BC547" x="10.16" y="5.08" smashed="yes" rot="R90">
 <attribute name="NAME" x="11.43" y="6.35" size="0.8128" layer="25" ratio="10" rot="R180" align="center"/>
@@
 <attribute name="VALUE" x="22.86" y="6.35" size="0.6096" layer="27" ratio="10" rot="R180" align="center"/>
 </element>
-<element name="R6" library="r" package="0202/7" value="1k" x="11.43" y="2.54"/>
+<element name="R6" library="r" package="0202/7" value="1kΩ" x="11.43" y="2.54"/>
 <element name="J2" library="pinconn" package="PIC-UART-X" value="PIC-UART-X" x="27.94" y="6.35" smashed="yes" rot="R180">
 <attribute name="NAME" x="27.94" y="1.016" size="0.8128" layer="25" align="top-center"/>
