File: eagle/RS232_NPN_PNP_FTDI232.brd (EAGLE design)
At the start: 14 parts, among them J1 FTDI232-BO-R, J2 PIC-UART-MCLR, T1 BC547, T2 BC557, T3 BC547

Commit message: ...
Parts:
- R1, R4, R6: value 10k -> 10kΩ
- R2, R5: value 1k -> 1kΩ
- R3: value 4.7k -> 4.7kΩ
- R7: value 470 -> 470Ω
Changed lines of the file:
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@@
 <elements>
 <element name="D1" library="d" package="DO34-5" value="1N4148" x="17.78" y="10.16"/>
-<element name="R1" library="r" package="0202/5" value="10k" x="12.7" y="7.62" rot="R180"/>
-<element name="R2" library="r" package="0202/10" value="1k" x="15.24" y="5.08" rot="R180"/>
-<element name="R3" library="r" package="0202/5" value="4.7k" x="20.32" y="7.62"/>
-<element name="R4" library="r" package="0202/7-V" value="10k" x="25.4" y="11.43" rot="R180"/>
-<element name="R5" library="r" package="0202/5-V" value="1k" x="27.94" y="10.16"/>
+<element name="R1" library="r" package="0202/5" value="10kΩ" x="12.7" y="7.62" rot="R180"/>
+<element name="R2" library="r" package="0202/10" value="1kΩ" x="15.24" y="5.08" rot="R180"/>
+<element name="R3" library="r" package="0202/5" value="4.7kΩ" x="20.32" y="7.62"/>
+<element name="R4" library="r" package="0202/7-V" value="10kΩ" x="25.4" y="11.43" rot="R180"/>
+<element name="R5" library="r" package="0202/5-V" value="1kΩ" x="27.94" y="10.16"/>
 <element name="T2" library="t" package="TO92-CBE" value="BC557" x="25.4" y="5.08" smashed="yes" rot="R90">
 <attribute name="NAME" x="24.384" y="6.35" size="0.8128" layer="25" ratio="10" rot="R180" align="center"/>
@@
 <attribute name="NAME" x="5.08" y="16.383" size="0.8128" layer="25" ratio="10" align="bottom-center"/>
 </element>
-<element name="R6" library="r" package="0202/7-V" value="10k" x="5.08" y="6.35" rot="R180"/>
+<element name="R6" library="r" package="0202/7-V" value="10kΩ" x="5.08" y="6.35" rot="R180"/>
 <element name="T3" library="t" package="TO92-CBE" value="BC547" x="10.16" y="12.7" smashed="yes" rot="R180">
 <attribute name="NAME" x="9.144" y="13.97" size="0.8128" layer="25" ratio="10" align="center"/>
@@
 <attribute name="NAME" x="31.242" y="3.048" size="0.8128" layer="25" align="top-left"/>
 </element>
-<element name="R7" library="r" package="0202/7-V" value="470" x="7.62" y="6.35" rot="R180"/>
+<element name="R7" library="r" package="0202/7-V" value="470Ω" x="7.62" y="6.35" rot="R180"/>
 </elements>
 <signals>
