File: eagle/RS232_NPN_PNP_FTDI_PowerSel.brd (EAGLE design)
At the start: 11 parts, among them J1 FTDI232-BO-5P-L, J2 PIC-UART, SW1 SL-SW-1P-2T-JPSW, T1 BC547, T2 BC557

Commit message: ...
Parts:
- R1, R4: value 10k -> 10kΩ
- R2, R5: value 1k -> 1kΩ
- R3: value 4.7k -> 4.7kΩ
Changed lines of the file:
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@@
 <elements>
 <element name="D1" library="d" package="DO34-5" value="1N4148" x="17.78" y="10.16"/>
-<element name="R1" library="r" package="0202/5-V" value="10k" x="2.54" y="7.62"/>
-<element name="R2" library="r" package="0202/5" value="1k" x="7.62" y="5.08" rot="R180"/>
-<element name="R3" library="r" package="0202/5-V" value="4.7k" x="10.16" y="10.16"/>
-<element name="R4" library="r" package="0202/5" value="10k" x="15.24" y="5.08" rot="R180"/>
-<element name="R5" library="r" package="0202/5-V" value="1k" x="20.32" y="5.08"/>
+<element name="R1" library="r" package="0202/5-V" value="10kΩ" x="2.54" y="7.62"/>
+<element name="R2" library="r" package="0202/5" value="1kΩ" x="7.62" y="5.08" rot="R180"/>
+<element name="R3" library="r" package="0202/5-V" value="4.7kΩ" x="10.16" y="10.16"/>
+<element name="R4" library="r" package="0202/5" value="10kΩ" x="15.24" y="5.08" rot="R180"/>
+<element name="R5" library="r" package="0202/5-V" value="1kΩ" x="20.32" y="5.08"/>
 <element name="T2" library="t" package="TO92-CBE" value="BC557" x="12.7" y="2.54" smashed="yes" rot="R90">
 <attribute name="NAME" x="11.684" y="3.81" size="0.8128" layer="25" ratio="10" rot="R180" align="center"/>
