File: eagle/RS232_NPN_PNP_Negative_FTDI.sch (EAGLE design)
At the start: 11 parts, among them J1 FTDI232-BO, J2 PIC-UART, T1 BC547CBE, T2 BC547CBE

Commit message: ...
Parts:
- C1: value 10uF -> 10μF
- R1, R2, R3, R4, R5: value 10k -> 10kΩ
Changed lines of the file:
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@@
 <part name="T1" library="t" deviceset="BC547" device="CBE" value="BC547CBE"/>
 <part name="D1" library="d" deviceset="1N4148" device="34-5V" value="1N4148"/>
-<part name="R1" library="r" deviceset="R" device="0202/5-V" value="10k"/>
+<part name="R1" library="r" deviceset="R" device="0202/5-V" value="10kΩ"/>
 <part name="T2" library="t" deviceset="BC547" device="CBE" value="BC547CBE"/>
-<part name="R2" library="r" deviceset="R" device="0202/10-V" value="10k"/>
-<part name="R3" library="r" deviceset="R" device="0202/7-V" value="10k"/>
-<part name="R4" library="r" deviceset="R" device="0202/7" value="10k"/>
-<part name="R5" library="r" deviceset="R" device="0202/2V" value="10k"/>
+<part name="R2" library="r" deviceset="R" device="0202/10-V" value="10kΩ"/>
+<part name="R3" library="r" deviceset="R" device="0202/7-V" value="10kΩ"/>
+<part name="R4" library="r" deviceset="R" device="0202/7" value="10kΩ"/>
+<part name="R5" library="r" deviceset="R" device="0202/2V" value="10kΩ"/>
 <part name="GND1" library="supply1" deviceset="GND" device=""/>
-<part name="C1" library="c" deviceset="CPOL" device="E2,5-5/V" value="10uF"/>
+<part name="C1" library="c" deviceset="CPOL" device="E2,5-5/V" value="10μF"/>
 <part name="P+1" library="supply1" deviceset="VCC" device=""/>
 <part name="P+2" library="supply1" deviceset="VCC" device=""/>
