File: eagle/insider.brd (EAGLE design)
At the start: 71.1 x 66 mm, 30 parts, among them IC2 ACPL-827, IC3 ACPL-827, IC4 7805, J2 CONN-2P2P/V, J4 COMPORT-6PIN-NEW, J5 CONN-2P2P/V, J6 CONN-2P2P/V, SW1 PB-1P-1T

Commit message: ...
Parts:
- C3, C4, C5: value 1uF -> 1μF
- R1, R2: value 22 -> 22Ω
- R10, R11, R12: value 1K5 -> 1.5kΩ
- R3: value 10K -> 10kΩ
- R4: value 100 -> 100Ω
- R5, R6: value 4K7 -> 4.7kΩ
- R7: value 1K -> 1kΩ
- R8: value 750 -> 750Ω
- R9: value 2K -> 2kΩ
Changed lines of the file:
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@@
         <element name="C1" library="c" package="C025-020X036" value="22P" x="60.96" y="43.18" />
         <element name="C2" library="c" package="C025-020X036" value="22P" x="60.96" y="38.1" />
-        <element name="C3" library="c" package="E2.5-4/V" value="1uF" x="22.86" y="7.62" rot="R180" />
-        <element name="C4" library="c" package="E2.5-4/V" value="1uF" x="43.18" y="10.16" rot="R90" />
-        <element name="C5" library="c" package="E2.5-4/V" value="1uF" x="33.02" y="55.88" />
+        <element name="C3" library="c" package="E2.5-4/V" value="1μF" x="22.86" y="7.62" rot="R180" />
+        <element name="C4" library="c" package="E2.5-4/V" value="1μF" x="43.18" y="10.16" rot="R90" />
+        <element name="C5" library="c" package="E2.5-4/V" value="1μF" x="33.02" y="55.88" />
         <element name="D1" library="d" package="DO34-5V" value="1N414834-5V" x="35.56" y="15.24" rot="R90" />
         <element name="D2" library="d" package="LED3MM" value="LED" x="53.34" y="59.69" rot="R270" />
@@
         <element name="IC4" library="ic" package="TO220" value="7805" x="34.29" y="7.62" rot="R90" />
         <element name="J4" library="pinconn" package="RS232-6PIN-NEW" value="COMPORT-6PIN-NEW" x="13.97" y="26.67" />
-        <element name="R1" library="r" package="0204/10" value="22" x="53.34" y="33.02" />
-        <element name="R10" library="r" package="0204/10" value="1K5" x="10.16" y="22.86" rot="R270" />
-        <element name="R11" library="r" package="0204/10" value="1K5" x="22.86" y="22.86" rot="R180" />
-        <element name="R12" library="r" package="0204/10" value="1K5" x="10.16" y="35.56" rot="R270" />
-        <element name="R2" library="r" package="0204/10" value="22" x="53.34" y="30.48" />
-        <element name="R3" library="r" package="0204/10" value="10K" x="48.26" y="22.86" rot="R180" />
-        <element name="R4" library="r" package="0204/15" value="100" x="33.02" y="30.48" rot="R90" />
-        <element name="R5" library="r" package="0204/10" value="4K7" x="48.26" y="50.8" rot="R270" />
-        <element name="R6" library="r" package="0204/10" value="4K7" x="53.34" y="50.8" rot="R270" />
-        <element name="R7" library="r" package="0204/10" value="1K" x="38.1" y="60.96" rot="R180" />
-        <element name="R8" library="r" package="0204/12" value="750" x="46.99" y="17.78" rot="R180" />
-        <element name="R9" library="r" package="0204/12" value="2K" x="46.99" y="20.32" rot="R180" />
+        <element name="R1" library="r" package="0204/10" value="22Ω" x="53.34" y="33.02" />
+        <element name="R10" library="r" package="0204/10" value="1.5kΩ" x="10.16" y="22.86" rot="R270" />
+        <element name="R11" library="r" package="0204/10" value="1.5kΩ" x="22.86" y="22.86" rot="R180" />
+        <element name="R12" library="r" package="0204/10" value="1.5kΩ" x="10.16" y="35.56" rot="R270" />
+        <element name="R2" library="r" package="0204/10" value="22Ω" x="53.34" y="30.48" />
+        <element name="R3" library="r" package="0204/10" value="10kΩ" x="48.26" y="22.86" rot="R180" />
+        <element name="R4" library="r" package="0204/15" value="100Ω" x="33.02" y="30.48" rot="R90" />
+        <element name="R5" library="r" package="0204/10" value="4.7kΩ" x="48.26" y="50.8" rot="R270" />
+        <element name="R6" library="r" package="0204/10" value="4.7kΩ" x="53.34" y="50.8" rot="R270" />
+        <element name="R7" library="r" package="0204/10" value="1kΩ" x="38.1" y="60.96" rot="R180" />
+        <element name="R8" library="r" package="0204/12" value="750Ω" x="46.99" y="17.78" rot="R180" />
+        <element name="R9" library="r" package="0204/12" value="2kΩ" x="46.99" y="20.32" rot="R180" />
         <element name="SW1" library="sw" package="PB-1P1T" value="PB-1P-1T" x="25.4" y="15.24" rot="R180" />
         <element name="U$4" library="mcu" package="DIL18-3/V" value="PIC16F628A/V" x="41.91" y="35.56" />
