File: eagle/pickit2.sch (EAGLE design)
At the start: 52 parts, among them IC1 PIC18F2550, IC2 MCP601P, J1 PN61729-S, J3 PIC-ICSP-ICSP, Q1 BS250P, Q2 2N7000, Q3 2N7000, Q5 2N7000, Q6 BS250P, Q7 2N7000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

Commit message: ...
Parts:
- C5, C8: value 10uF -> 10μF
- C9: value 47uF -> 47μF
- L1: value 680uH -> 680μH
- R1, R10, R16, R3, R4, R5: value 10K -> 10kΩ
- R11: value 100 -> 100Ω
- R12: value 1K -> 1kΩ
- R13, R17, R18, R8: value 4.7K -> 4.7kΩ
- R14, R15: value 43 -> 43Ω
- R2, R6, R7: value 470 -> 470Ω
- R9: value 2.7K -> 2.7kΩ
Changed lines of the file:
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@@
 <part name="X1" library="q" deviceset="CRYSTAL" device="HC49" value="20Mhz"/>
 <part name="P+9" library="supply1" deviceset="+5V" device=""/>
-<part name="L1" library="inductors" deviceset="82114R" device="M" value="680uH"/>
-<part name="R8" library="r" deviceset="R" device="0204/10" value="4.7K"/>
+<part name="L1" library="inductors" deviceset="82114R" device="M" value="680μH"/>
+<part name="R8" library="r" deviceset="R" device="0204/10" value="4.7kΩ" />
 <part name="D2" library="diode" deviceset="BAT42" device="M" value="BAT85"/>
 <part name="Q3" library="t" deviceset="2N7000" device="" value="2N7000"/>
@@
 <part name="GND7" library="supply1" deviceset="GND" device=""/>
 <part name="GND8" library="supply1" deviceset="GND" device=""/>
-<part name="R4" library="r" deviceset="R-H" device="0204/10" value="10K"/>
-<part name="R1" library="r" deviceset="R-H" device="0204/10" value="10K"/>
+<part name="R4" library="r" deviceset="R-H" device="0204/10" value="10kΩ" />
+<part name="R1" library="r" deviceset="R-H" device="0204/10" value="10kΩ" />
 <part name="GND9" library="supply1" deviceset="GND" device=""/>
 <part name="GND10" library="supply1" deviceset="GND" device=""/>
 <part name="GND11" library="supply1" deviceset="GND" device=""/>
-<part name="R16" library="r" deviceset="R-H" device="0204/10" value="10K"/>
+<part name="R16" library="r" deviceset="R-H" device="0204/10" value="10kΩ" />
 <part name="GND13" library="supply1" deviceset="GND" device=""/>
 <part name="GND14" library="supply1" deviceset="GND" device=""/>
@@
 <part name="GND16" library="supply1" deviceset="GND" device=""/>
 <part name="IC2" library="linear" deviceset="MCP601" device="M" value="MCP601P"/>
-<part name="R10" library="r" deviceset="R" device="0204/10" value="10K"/>
-<part name="R9" library="r" deviceset="R" device="0204/10" value="2.7K"/>
-<part name="R11" library="r" deviceset="R" device="0204/10" value="100"/>
-<part name="R12" library="r" deviceset="R" device="0204/10" value="1K"/>
-<part name="R15" library="r" deviceset="R-H" device="0204/10" value="43"/>
-<part name="R14" library="r" deviceset="R-H" device="0204/10" value="43"/>
-<part name="R13" library="r" deviceset="R-H" device="0204/10" value="4.7K"/>
-<part name="R17" library="r" deviceset="R" device="0204/10" value="4.7K"/>
-<part name="R18" library="r" deviceset="R" device="0204/10" value="4.7K"/>
-<part name="R3" library="r" deviceset="R" device="0204/10" value="10K"/>
-<part name="R7" library="r" deviceset="R" device="0204/10" value="470"/>
-<part name="R6" library="r" deviceset="R" device="0204/10" value="470"/>
-<part name="R2" library="r" deviceset="R" device="0204/10" value="470"/>
-<part name="R5" library="r" deviceset="R" device="0204/10" value="10K"/>
+<part name="R10" library="r" deviceset="R" device="0204/10" value="10kΩ" />
+<part name="R9" library="r" deviceset="R" device="0204/10" value="2.7kΩ" />
+<part name="R11" library="r" deviceset="R" device="0204/10" value="100Ω"/>
+<part name="R12" library="r" deviceset="R" device="0204/10" value="1kΩ" />
+<part name="R15" library="r" deviceset="R-H" device="0204/10" value="43Ω"/>
+<part name="R14" library="r" deviceset="R-H" device="0204/10" value="43Ω"/>
+<part name="R13" library="r" deviceset="R-H" device="0204/10" value="4.7kΩ" />
+<part name="R17" library="r" deviceset="R" device="0204/10" value="4.7kΩ" />
+<part name="R18" library="r" deviceset="R" device="0204/10" value="4.7kΩ" />
+<part name="R3" library="r" deviceset="R" device="0204/10" value="10kΩ" />
+<part name="R7" library="r" deviceset="R" device="0204/10" value="470Ω"/>
+<part name="R6" library="r" deviceset="R" device="0204/10" value="470Ω"/>
+<part name="R2" library="r" deviceset="R" device="0204/10" value="470Ω"/>
+<part name="R5" library="r" deviceset="R" device="0204/10" value="10kΩ" />
 <part name="GND1" library="supply1" deviceset="GND" device=""/>
 <part name="J1" library="con-berg" deviceset="PN61729-S" device="" value=""/>
@@
 <part name="C4" library="c" deviceset="C" device="050-025X075/V" value="100nF"/>
 <part name="J3" library="pinconn" deviceset="PIC-ICSP" device="-ICSP"/>
-<part name="C8" library="c" deviceset="CPOL" device="E2.5-5" value="10uF"/>
-<part name="C9" library="c" deviceset="CPOL" device="E2.5-5" value="47uF"/>
-<part name="C5" library="c" deviceset="CPOL" device="E2.5-5" value="10uF"/>
+<part name="C8" library="c" deviceset="CPOL" device="E2.5-5" value="10μF"/>
+<part name="C9" library="c" deviceset="CPOL" device="E2.5-5" value="47μF"/>
+<part name="C5" library="c" deviceset="CPOL" device="E2.5-5" value="10μF"/>
 <part name="C6" library="c" deviceset="C" device="050-025X075/V" value="470nF"/>
 </parts>
