File: eagle/PIC18F25k50-USB+ICSP-Board.brd (EAGLE design)
At the start: 18 parts, among them J1 PIC-ICSP-ICSP, J2 USB-PRINT, J3 RA[0..4], J4 RC[0..3], J5 PWR+SCI+USB, J6 RB[0..7], SW1 PB-1P-1T

Commit message: ...
Parts:
- C5: value 100uF -> 100μF
- R1, R5: value 330 -> 330Ω
- R2, R3: value 100 -> 100Ω
- R4: value 10k -> 10kΩ
Changed lines of the file:
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@@
 <element name="C2" library="c" package="C025-015X024" value="100n" x="25.4" y="31.75"/>
 <element name="J2" library="usb" package="USB-B-PRINT" value="USB-PRINT" x="17.78" y="7.62" rot="R90"/>
-<element name="R1" library="r" package="0204/10" value="330" x="5.08" y="35.56" rot="R270"/>
+<element name="R1" library="r" package="0204/10" value="330Ω" x="5.08" y="35.56" rot="R270"/>
 <element name="LED1" library="led" package="LED5MM" value="" x="7.62" y="34.29" rot="R90"/>
-<element name="C5" library="c" package="E2,5-5" value="100uF" x="30.48" y="11.43" rot="R90"/>
+<element name="C5" library="c" package="E2,5-5" value="100μF" x="30.48" y="11.43" rot="R90"/>
 <element name="J4" library="pinconn" package="CONN-4P" value="RC[0..3]" x="2.54" y="24.13" rot="R270"/>
 <element name="J5" library="pinconn" package="CONN-6P" value="PWR+SCI+USB" x="35.56" y="26.67" rot="R90"/>
 <element name="J6" library="pinconn" package="CONN-8P" value="RB[0..7]" x="35.56" y="35.56" rot="R90"/>
 <element name="J3" library="pinconn" package="CONN-5P-N" value="RA[0..4]" x="2.54" y="45.72" rot="R270"/>
-<element name="R2" library="r" package="0204/7-V" value="100" x="27.94" y="57.15"/>
-<element name="R3" library="r" package="0204/7-V" value="100" x="25.4" y="54.61"/>
+<element name="R2" library="r" package="0204/7-V" value="100Ω" x="27.94" y="57.15"/>
+<element name="R3" library="r" package="0204/7-V" value="100Ω" x="25.4" y="54.61"/>
 <element name="U$1" library="mcu" package="PIC18F2550-V" value="PIC18F2550-I/SPLABEL" x="19.05" y="38.1"/>
-<element name="R4" library="r" package="0204/10" value="10k" x="15.24" y="55.88"/>
+<element name="R4" library="r" package="0204/10" value="10kΩ" x="15.24" y="55.88"/>
 <element name="SW1" library="sw" package="PB-1P1T" value="PB-1P-1T" x="2.54" y="58.42" rot="R270"/>
-<element name="R5" library="r" package="0204/10" value="330" x="15.24" y="58.42" rot="R180"/>
+<element name="R5" library="r" package="0204/10" value="330Ω" x="15.24" y="58.42" rot="R180"/>
 <element name="LED2" library="led" package="LED5MM" value="" x="7.62" y="62.23" rot="R90"/>
 </elements>

Commit message: ...
Parts:
- J1: value PIC-ICSP-ICSP -> PIC-ICSPICSP
- J3: device pinconn:CONN-5P-N -> pinconn:CONN-5P
- moved J5 6.35 mm to (35.6, 20.3)
- moved J3 5.08 mm to (2.54, 50.8)
- moved J4 3.81 mm to (2.54, 27.9)
- moved C2 2.54 mm to (27.9, 31.8), turned to 270 degrees
Routing:
- net VCC: track 86.4 -> 81.3 mm
Changed lines of the file:
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@@
 </autorouter>
 <elements>
-<element name="J1" library="pinconn" package="PIC-ICSP" value="PIC-ICSP-ICSP" x="17.78" y="63.5"/>
+<element name="J1" library="pinconn" package="PIC-ICSP" value="PIC-ICSPICSP" x="17.78" y="63.5"/>
 <element name="C1" library="c" package="C050-030X075" value="330n" x="10.16" y="17.78" rot="R270"/>
-<element name="C2" library="c" package="C025-015X024" value="100n" x="25.4" y="31.75"/>
+<element name="C2" library="c" package="C025-015X024" value="100n" x="27.94" y="31.75" rot="R270"/>
 <element name="J2" library="usb" package="USB-B-PRINT" value="USB-PRINT" x="17.78" y="7.62" rot="R90"/>
 <element name="R1" library="r" package="0204/10" value="330Ω" x="5.08" y="35.56" rot="R270"/>
 <element name="LED1" library="led" package="LED5MM" value="" x="7.62" y="34.29" rot="R90"/>
 <element name="C5" library="c" package="E2,5-5" value="100μF" x="30.48" y="11.43" rot="R90"/>
-<element name="J4" library="pinconn" package="CONN-4P" value="RC[0..3]" x="2.54" y="24.13" rot="R270"/>
-<element name="J5" library="pinconn" package="CONN-6P" value="PWR+SCI+USB" x="35.56" y="26.67" rot="R90"/>
+<element name="J4" library="pinconn" package="CONN-4P" value="RC[0..3]" x="2.54" y="27.94" rot="R270"/>
+<element name="J5" library="pinconn" package="CONN-6P" value="PWR+SCI+USB" x="35.56" y="20.32" rot="R90"/>
 <element name="J6" library="pinconn" package="CONN-8P" value="RB[0..7]" x="35.56" y="35.56" rot="R90"/>
-<element name="J3" library="pinconn" package="CONN-5P-N" value="RA[0..4]" x="2.54" y="45.72" rot="R270"/>
+<element name="J3" library="pinconn" package="CONN-5P" value="RA[0..4]" x="2.54" y="50.8" rot="R270"/>
 <element name="R2" library="r" package="0204/7-V" value="100Ω" x="27.94" y="57.15"/>
 <element name="R3" library="r" package="0204/7-V" value="100Ω" x="25.4" y="54.61"/>
@@
 <contactref element="J5" pad="5"/>
 <wire x1="35.56" y1="30.48" x2="33.02" y2="30.48" width="0.8128" layer="16"/>
-<wire x1="33.02" y1="30.48" x2="25.4" y2="30.48" width="0.8128" layer="16"/>
+<wire x1="33.02" y1="30.48" x2="27.94" y2="30.48" width="0.8128" layer="16"/>
 <via x="33.02" y="30.48" extent="1-16" drill="0.6" shape="square"/>
 <wire x1="33.02" y1="30.48" x2="33.02" y2="17.78" width="0.8128" layer="1"/>
@@
 <contactref element="U$1" pad="8"/>
 <wire x1="15.24" y1="35.56" x2="17.78" y2="35.56" width="0.8128" layer="16"/>
-<wire x1="22.86" y1="30.48" x2="25.4" y2="30.48" width="0.8128" layer="16"/>
+<wire x1="22.86" y1="30.48" x2="27.94" y2="30.48" width="0.8128" layer="16"/>
 <wire x1="17.78" y1="30.48" x2="22.86" y2="30.48" width="0.8128" layer="16"/>
 <contactref element="SW1" pad="2"/>
@@
 <contactref element="U$1" pad="20"/>
 <wire x1="30.48" y1="33.02" x2="20.32" y2="33.02" width="0.8128" layer="16"/>
-<wire x1="35.56" y1="33.02" x2="25.4" y2="33.02" width="0.8128" layer="16"/>
-<wire x1="25.4" y1="33.02" x2="30.48" y2="33.02" width="0.8128" layer="16"/>
+<wire x1="35.56" y1="33.02" x2="27.94" y2="33.02" width="0.8128" layer="16"/>
+<wire x1="27.94" y1="33.02" x2="30.48" y2="33.02" width="0.8128" layer="16"/>
 <via x="30.48" y="33.02" extent="1-16" drill="0.381"/>
 <wire x1="30.48" y1="33.02" x2="30.48" y2="17.78" width="0.8128" layer="1"/>
@@
 <wire x1="20.32" y1="58.42" x2="20.32" y2="33.02" width="0.8128" layer="16"/>
 <wire x1="20.32" y1="58.42" x2="20.32" y2="55.88" width="0" layer="19" extent="1-1"/>
-<wire x1="22.86" y1="33.02" x2="25.4" y2="33.02" width="0" layer="19" extent="1-1"/>
+<wire x1="22.86" y1="33.02" x2="20.32" y2="33.02" width="0" layer="19" extent="16-16"/>
 </signal>
 <signal name="N$1">
