File: eagle/JDM2_2-Voltage.brd (EAGLE design)
At the start: 19 parts, among them J1 COMPORT-6PIN, J2 PIC-ICSPICSP, SW1 SL-SW-2P-2T-S, T1 BC547CBE-A, T2 BC547CBE

Commit message: ...
Parts:
- C1: value 100uF -> 100μF
- C2: value 22uF -> 22μF
- R1: value 10k -> 10kΩ
- R2: value 1.5k -> 1.5kΩ
- R3: value 100 -> 100Ω
Changed lines of the file:
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@@
 </autorouter>
 <elements>
-<element name="C1" library="c" package="E5-4" value="100uF" x="15.24" y="25.4" rot="R180"/>
-<element name="C2" library="c" package="E2,5-4" value="22uF" x="11.43" y="17.78" rot="R180"/>
+<element name="C1" library="c" package="E5-4" value="100μF" x="15.24" y="25.4" rot="R180"/>
+<element name="C2" library="c" package="E2,5-4" value="22μF" x="11.43" y="17.78" rot="R180"/>
 <element name="D1" library="d" package="DO34-5" value="1N4148" x="15.24" y="20.32" rot="R180"/>
 <element name="D4" library="d" package="DO34Z5" value="Z=8.1V" x="20.32" y="22.86" rot="R90"/>
@@
 <attribute name="VALUE" x="21.971" y="33.655" size="1.27" layer="27" ratio="10" rot="R90"/>
 </element>
-<element name="R1" library="r" package="0202/7" value="10k" x="8.89" y="30.48" rot="R270"/>
-<element name="R2" library="r" package="0202/7" value="1.5k" x="8.89" y="33.02" rot="R90"/>
+<element name="R1" library="r" package="0202/7" value="10kΩ" x="8.89" y="30.48" rot="R270"/>
+<element name="R2" library="r" package="0202/7" value="1.5kΩ" x="8.89" y="33.02" rot="R90"/>
 <element name="T1" library="t" package="TO92-CBE-A" value="BC547CBE-A" x="5.08" y="17.78"/>
 <element name="T2" library="t" package="TO92-CBE" value="BC547CBE" x="2.54" y="30.48"/>
-<element name="R3" library="r" package="0202/5" value="100" x="0" y="25.4"/>
+<element name="R3" library="r" package="0202/5" value="100Ω" x="0" y="25.4"/>
 <element name="J2" library="pinconn" package="PIC-ICSP" value="PIC-ICSPICSP" x="7.62" y="2.54" rot="R180"/>
 <element name="SW1" library="sw" package="SLSW-2P2T-H" value="SL-SW-2P-2T-S" x="19.05" y="10.16" rot="R180"/>

Commit message: ...
Other:
- board outline added: 27.9 x 38.1 mm
Changed lines of the file:
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@@
 <description>JDM2 with selectable Dual-Voltage</description>
 <plain>
-<wire x1="-2.54" y1="0" x2="25.4" y2="0" width="0" layer="47"/>
-<wire x1="25.4" y1="0" x2="25.4" y2="38.1" width="0" layer="47"/>
-<wire x1="25.4" y1="38.1" x2="-2.54" y2="38.1" width="0" layer="47"/>
-<wire x1="-2.54" y1="38.1" x2="-2.54" y2="0" width="0" layer="47"/>
+<wire x1="-2.54" y1="0" x2="25.4" y2="0" width="0" layer="20"/>
+<wire x1="25.4" y1="0" x2="25.4" y2="38.1" width="0" layer="20"/>
+<wire x1="25.4" y1="38.1" x2="-2.54" y2="38.1" width="0" layer="20"/>
+<wire x1="-2.54" y1="38.1" x2="-2.54" y2="0" width="0" layer="20"/>
 </plain>
 <attributes>
