File: eagle/JDM2_2-Voltage_Pretty.brd (EAGLE design)
At the start: 18 parts, among them J1 COMPORT-6PIN, J2 PIC-ICSPICSP, SW2 SL-SW-2P-2T-SV, T1 BC547, T2 BC547

Commit message: ...
Parts:
- C1: value 100uF -> 100μF
- C2: value 22uF -> 22μF
- R1: value 10k -> 10kΩ
- R2: value 1.5k -> 1.5kΩ
- R3: value 100 -> 100Ω
Changed lines of the file:
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@@
 </autorouter>
 <elements>
-<element name="C1" library="c" package="E2,5-4" value="100uF" x="21.59" y="2.54" rot="R90"/>
-<element name="C2" library="c" package="E2,5-5" value="22uF" x="34.29" y="2.54"/>
+<element name="C1" library="c" package="E2,5-4" value="100μF" x="21.59" y="2.54" rot="R90"/>
+<element name="C2" library="c" package="E2,5-5" value="22μF" x="34.29" y="2.54"/>
 <element name="D1" library="d" package="DO34-5V" value="1N4148" x="15.24" y="0" rot="R270"/>
 <element name="D2" library="d" package="DO34-2,5-A" value="1N4148" x="5.08" y="1.27" rot="R90"/>
@@
 <attribute name="NAME" x="40.64" y="1.27" size="0.8128" layer="25" rot="R90" align="top-left"/>
 </element>
-<element name="R1" library="r" package="0202/7-V" value="10k" x="35.56" y="8.89" rot="R180"/>
-<element name="R2" library="r" package="0202/7-V" value="1.5k" x="2.54" y="8.89" rot="R180"/>
-<element name="R3" library="r" package="0202/5" value="100" x="40.64" y="17.78" rot="R90"/>
+<element name="R1" library="r" package="0202/7-V" value="10kΩ" x="35.56" y="8.89" rot="R180"/>
+<element name="R2" library="r" package="0202/7-V" value="1.5kΩ" x="2.54" y="8.89" rot="R180"/>
+<element name="R3" library="r" package="0202/5" value="100Ω" x="40.64" y="17.78" rot="R90"/>
 <element name="T1" library="t" package="TO92-CBE" value="BC547" x="10.16" y="2.54" rot="R270"/>
 <element name="T2" library="t" package="TO92-CBE-A" value="BC547" x="35.56" y="12.7" rot="R90"/>

Commit message: ...
Other:
- board outline added: 45.7 x 25.4 mm
Changed lines of the file:
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@@
 <description>JDM2 with selectable Dual-Voltage</description>
 <plain>
-<wire x1="-1.27" y1="-1.27" x2="44.45" y2="-1.27" width="0.6096" layer="47"/>
-<wire x1="44.45" y1="-1.27" x2="44.45" y2="24.13" width="0" layer="47"/>
-<wire x1="44.45" y1="24.13" x2="-1.27" y2="24.13" width="0" layer="47"/>
-<wire x1="-1.27" y1="24.13" x2="-1.27" y2="-1.27" width="0" layer="47"/>
+<wire x1="-1.27" y1="-1.27" x2="44.45" y2="-1.27" width="0.6096" layer="20"/>
+<wire x1="44.45" y1="-1.27" x2="44.45" y2="24.13" width="0" layer="20"/>
+<wire x1="44.45" y1="24.13" x2="-1.27" y2="24.13" width="0" layer="20"/>
+<wire x1="-1.27" y1="24.13" x2="-1.27" y2="-1.27" width="0" layer="20"/>
 </plain>
 <attributes>
