File: eagle/JDM2_Basic.brd (EAGLE design)
At the start: 16 parts, among them J1 COMPORT-6PIN, T1 BC547CBE-A, T2 BC547CBE

Commit message: ...
Parts:
- C1: value 100uF -> 100μF
- C2: value 22uF -> 22μF
- R1: value 10k -> 10kΩ
- R2: value 1.5k -> 1.5kΩ
- R3: value 100 -> 100Ω
Changed lines of the file:
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@@
 </autorouter>
 <elements>
-<element name="C1" library="c" package="E5-4" value="100uF" x="20.32" y="7.62" rot="R270"/>
-<element name="C2" library="c" package="E2,5-4" value="22uF" x="8.89" y="5.08" rot="R180"/>
+<element name="C1" library="c" package="E5-4" value="100μF" x="20.32" y="7.62" rot="R270"/>
+<element name="C2" library="c" package="E2,5-4" value="22μF" x="8.89" y="5.08" rot="R180"/>
 <element name="D1" library="d" package="DO34-2,5-A" value="1N4148" x="27.94" y="3.81" rot="R90"/>
 <element name="D4" library="d" package="DO34Z5" value="Z=8.1V" x="15.24" y="10.16" smashed="yes" rot="R270">
@@
 <attribute name="VALUE" x="17.145" y="14.351" size="1.27" layer="27" ratio="10" rot="R180"/>
 </element>
-<element name="R1" library="r" package="0202/5" value="10k" x="7.62" y="10.16" rot="R180"/>
-<element name="R2" library="r" package="0202/7" value="1.5k" x="5.08" y="8.89"/>
+<element name="R1" library="r" package="0202/5" value="10kΩ" x="7.62" y="10.16" rot="R180"/>
+<element name="R2" library="r" package="0202/7" value="1.5kΩ" x="5.08" y="8.89"/>
 <element name="T1" library="t" package="TO92-CBE-A" value="BC547CBE-A" x="25.4" y="10.16" rot="R90"/>
 <element name="T2" library="t" package="TO92-CBE" value="BC547CBE" x="7.62" y="15.24" rot="R90"/>
-<element name="R3" library="r" package="0202/5" value="100" x="12.7" y="17.78" rot="R90"/>
+<element name="R3" library="r" package="0202/5" value="100Ω" x="12.7" y="17.78" rot="R90"/>
 <element name="U$5" library="pinconn" package="PIC-ICSP" value="PIC-ICSPICSP" x="33.02" y="10.16" rot="R90"/>
 </elements>

Commit message: ...
Other:
- board outline added: 35.5 x 20 mm
Changed lines of the file:
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@@
 <description>JDM2 Basic Design</description>
 <plain>
-<wire x1="0" y1="0" x2="35.54" y2="0" width="0" layer="47"/>
-<wire x1="35.54" y1="0" x2="35.54" y2="19.99" width="0" layer="47"/>
-<wire x1="35.54" y1="19.99" x2="0" y2="19.99" width="0" layer="47"/>
-<wire x1="0" y1="19.99" x2="0" y2="0" width="0" layer="47"/>
+<wire x1="0" y1="0" x2="35.54" y2="0" width="0" layer="20"/>
+<wire x1="35.54" y1="0" x2="35.54" y2="19.99" width="0" layer="20"/>
+<wire x1="35.54" y1="19.99" x2="0" y2="19.99" width="0" layer="20"/>
+<wire x1="0" y1="19.99" x2="0" y2="0" width="0" layer="20"/>
 </plain>
 <attributes>
