File: eagle/JDM2_Basic_2.brd (EAGLE design)
At the start: 16 parts, among them J1 COMPORT-6PIN, J2 PIC-ICSPICSP, T1 BC547CBE, T2 BC547CBE

Commit message: ...
Parts:
- C1: value 100uF -> 100μF
- C2: value 22uF -> 22μF
- R1: value 10k -> 10kΩ
- R2: value 1.5k -> 1.5kΩ
- R3: value 100 -> 100Ω
Changed lines of the file:
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@@
 </autorouter>
 <elements>
-<element name="C1" library="c" package="E5-4" value="100uF" x="11.43" y="15.24"/>
-<element name="C2" library="c" package="E2,5-4" value="22uF" x="13.97" y="21.59" rot="R90"/>
+<element name="C1" library="c" package="E5-4" value="100μF" x="11.43" y="15.24"/>
+<element name="C2" library="c" package="E2,5-4" value="22μF" x="13.97" y="21.59" rot="R90"/>
 <element name="D1" library="d" package="DO34-2,5-A" value="1N4148" x="15.24" y="12.7" rot="R180"/>
 <element name="D4" library="d" package="DO34Z7" value="Z=8.1V" x="7.62" y="20.32" smashed="yes">
@@
 <attribute name="VALUE" x="3.175" y="16.891" size="1.27" layer="27" ratio="10" rot="R180"/>
 </element>
-<element name="R1" library="r" package="0202/7" value="10k" x="7.62" y="22.86" rot="R270"/>
-<element name="R2" library="r" package="0202/7" value="1.5k" x="10.16" y="27.94" rot="R90"/>
+<element name="R1" library="r" package="0202/7" value="10kΩ" x="7.62" y="22.86" rot="R270"/>
+<element name="R2" library="r" package="0202/7" value="1.5kΩ" x="10.16" y="27.94" rot="R90"/>
 <element name="T1" library="t" package="TO92-CBE" value="BC547CBE" x="6.35" y="10.16"/>
 <element name="T2" library="t" package="TO92-CBE" value="BC547CBE" x="3.81" y="25.4" rot="R270"/>
-<element name="R3" library="r" package="0202/5" value="100" x="1.27" y="20.32"/>
+<element name="R3" library="r" package="0202/5" value="100Ω" x="1.27" y="20.32"/>
 <element name="J2" library="pinconn" package="PIC-ICSP" value="PIC-ICSPICSP" x="8.89" y="2.54" rot="R180"/>
 </elements>

Commit message: ...
Other:
- board outline added: 20.3 x 33 mm
Changed lines of the file:
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@@
 <description>JDM2 Basic Design</description>
 <plain>
-<wire x1="0" y1="0" x2="20.32" y2="0" width="0" layer="47"/>
-<wire x1="20.32" y1="0" x2="20.32" y2="33.02" width="0" layer="47"/>
-<wire x1="20.32" y1="33.02" x2="0" y2="33.02" width="0" layer="47"/>
-<wire x1="0" y1="33.02" x2="0" y2="0" width="0" layer="47"/>
+<wire x1="0" y1="0" x2="20.32" y2="0" width="0" layer="20"/>
+<wire x1="20.32" y1="0" x2="20.32" y2="33.02" width="0" layer="20"/>
+<wire x1="20.32" y1="33.02" x2="0" y2="33.02" width="0" layer="20"/>
+<wire x1="0" y1="33.02" x2="0" y2="0" width="0" layer="20"/>
 </plain>
 <attributes>
