File: eagle/JDM2_Basic_No_Top_Aligned.brd (EAGLE design)
At the start: 19 parts, among them J1 COMPORT-6PIN, T1 BC547CBE, T2 BC547CBE-A

Commit message: ...
Parts:
- C1: value 100uF -> 100μF
- C2: value 22uF -> 22μF
- R1: value 10k -> 10kΩ
- R2: value 1.5k -> 1.5kΩ
- R3: value 100 -> 100Ω
Changed lines of the file:
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@@
 </autorouter>
 <elements>
-<element name="C1" library="c" package="E5-4" value="100uF" x="88.9" y="17.78" rot="R180"/>
-<element name="C2" library="c" package="E2,5-4" value="22uF" x="48.26" y="19.05" rot="R90"/>
+<element name="C1" library="c" package="E5-4" value="100μF" x="88.9" y="17.78" rot="R180"/>
+<element name="C2" library="c" package="E2,5-4" value="22μF" x="48.26" y="19.05" rot="R90"/>
 <element name="D1" library="d" package="DO34-2,5-A" value="1N4148" x="83.82" y="16.51" rot="R90"/>
 <element name="D4" library="d" package="DO34Z7" value="Z=8.1V" x="81.28" y="16.51" rot="MR90"/>
@@
 <element name="J1" library="pinconn" package="RS232-6PIN" value="COMPORT-6PIN" x="43.18" y="15.24" rot="R90"/>
 <element name="D3" library="led" package="LED3MM" value="Vpp" x="90.17" y="12.7" rot="R180"/>
-<element name="R1" library="r" package="0202/5" value="10k" x="55.88" y="22.86" rot="R180"/>
-<element name="R2" library="r" package="0202/7" value="1.5k" x="45.72" y="21.59"/>
+<element name="R1" library="r" package="0202/5" value="10kΩ" x="55.88" y="22.86" rot="R180"/>
+<element name="R2" library="r" package="0202/7" value="1.5kΩ" x="45.72" y="21.59"/>
 <element name="T1" library="t" package="TO92-CBE" value="BC547CBE" x="88.9" y="22.86" rot="R270"/>
 <element name="T2" library="t" package="TO92-CBE-A" value="BC547CBE-A" x="55.88" y="25.4" rot="R90"/>
-<element name="R3" library="r" package="0202/2V" value="100" x="59.69" y="27.94" rot="R90"/>
+<element name="R3" library="r" package="0202/2V" value="100Ω" x="59.69" y="27.94" rot="R90"/>
 <element name="C3" library="c" package="C050-020X036" value="39pF" x="50.8" y="38.1"/>
 <element name="C4" library="c" package="C050-020X036" value="39pF" x="60.96" y="20.32"/>

Commit message: ...
Other:
- board outline added: 160 x 100 mm
Changed lines of the file:
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@@
 <description>JDM2 Basic Design</description>
 <plain>
-<wire x1="0" y1="0" x2="160" y2="0" width="0" layer="47"/>
-<wire x1="160" y1="0" x2="160" y2="100" width="0" layer="47"/>
-<wire x1="160" y1="100" x2="0" y2="100" width="0" layer="47"/>
-<wire x1="0" y1="100" x2="0" y2="0" width="0" layer="47"/>
+<wire x1="0" y1="0" x2="160" y2="0" width="0" layer="20"/>
+<wire x1="160" y1="0" x2="160" y2="100" width="0" layer="20"/>
+<wire x1="160" y1="100" x2="0" y2="100" width="0" layer="20"/>
+<wire x1="0" y1="100" x2="0" y2="0" width="0" layer="20"/>
 </plain>
 <attributes>
