File: eagle/JDM2_Low_Voltage.brd (EAGLE design)
At the start: 27 parts, among them J1 DUMMY, T1 BC547, T2 BC547, T3 2N7000

Commit message: ...
Parts:
- C1: value 100uF -> 100μF
- C2: value 22uF -> 22μF
- R1: value 10k -> 10kΩ
- R2: value 1.5k -> 1.5kΩ
- R4: value 1K -> 1kΩ
- R5: value 15K -> 15kΩ
- R6: value 4.7k -> 4.7kΩ
- R7: value 1k -> 1kΩ
Changed lines of the file:
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@@
 </autorouter>
 <elements>
-<element name="C1" library="rcl" package="E2,5-5" value="100uF" x="20.32" y="29.21" rot="R270"/>
-<element name="C2" library="rcl" package="E2,5-5" value="22uF" x="35.56" y="29.21" rot="R270"/>
+<element name="C1" library="rcl" package="E2,5-5" value="100μF" x="20.32" y="29.21" rot="R270"/>
+<element name="C2" library="rcl" package="E2,5-5" value="22μF" x="35.56" y="29.21" rot="R270"/>
 <element name="D1" library="JDM2" package="DO35-7" value="1N4148" x="15.24" y="31.75" rot="R270"/>
 <element name="D10" library="JDM2" package="DO35-2_54A" value="1N4148" x="44.45" y="30.48"/>
@@
 <element name="LED1" library="1dmf" package="LED5MM" value="Power" x="50.8" y="29.21" rot="R270"/>
 <element name="LED2" library="1dmf" package="LED5MM" value="Vpp" x="27.94" y="29.21" rot="R270"/>
-<element name="R1" library="JDM2" package="0207/10" value="10k" x="45.72" y="48.26" rot="R180"/>
-<element name="R2" library="JDM2" package="0204/7" value="1.5k" x="58.42" y="41.91" rot="R90"/>
-<element name="R4" library="JDM2" package="0207/10" value="1K" x="20.32" y="50.8" rot="R180"/>
-<element name="R5" library="JDM2" package="0207/10" value="15K" x="20.32" y="48.26" rot="R180"/>
-<element name="R6" library="JDM2" package="0204/7" value="4.7k" x="27.94" y="36.83" rot="R90"/>
-<element name="R7" library="JDM2" package="0204/7" value="1k" x="50.8" y="36.83" rot="R90"/>
+<element name="R1" library="JDM2" package="0207/10" value="10kΩ" x="45.72" y="48.26" rot="R180"/>
+<element name="R2" library="JDM2" package="0204/7" value="1.5kΩ" x="58.42" y="41.91" rot="R90"/>
+<element name="R4" library="JDM2" package="0207/10" value="1kΩ" x="20.32" y="50.8" rot="R180"/>
+<element name="R5" library="JDM2" package="0207/10" value="15kΩ" x="20.32" y="48.26" rot="R180"/>
+<element name="R6" library="JDM2" package="0204/7" value="4.7kΩ" x="27.94" y="36.83" rot="R90"/>
+<element name="R7" library="JDM2" package="0204/7" value="1kΩ" x="50.8" y="36.83" rot="R90"/>
 <element name="T1" library="JDM2" package="TO92-CBE" value="BC547" x="20.32" y="38.1" rot="R90"/>
 <element name="T2" library="JDM2" package="TO92-CBE" value="BC547" x="50.8" y="45.72" rot="R180"/>

Commit message: ...
Changed lines of the file:
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@@
 <board>
 <plain>
-<wire x1="0" y1="0" x2="160" y2="0" width="0" layer="47"/>
-<wire x1="160" y1="0" x2="160" y2="100" width="0" layer="47"/>
-<wire x1="160" y1="100" x2="0" y2="100" width="0" layer="47"/>
-<wire x1="0" y1="100" x2="0" y2="0" width="0" layer="47"/>
+<wire x1="0" y1="0" x2="160" y2="0" width="0" layer="20"/>
+<wire x1="160" y1="0" x2="160" y2="100" width="0" layer="20"/>
+<wire x1="160" y1="100" x2="0" y2="100" width="0" layer="20"/>
+<wire x1="0" y1="100" x2="0" y2="0" width="0" layer="20"/>
 </plain>
 <attributes>
