File: eagle/JDM2_NoDIL.brd (EAGLE design)
At the start: 24 parts, among them J1 DUMMY, T1 BC547, T2 BC547, T3 2N7000

Commit message: ...
Parts:
- C1: value 100uF -> 100μF
- C2: value 22uF -> 22μF
- R1: value 10k -> 10kΩ
- R2: value 1.5k -> 1.5kΩ
- R4: value 1K -> 1kΩ
- R5: value 15K -> 15kΩ
- R6: value 4.7k -> 4.7kΩ
- R7: value 1k -> 1kΩ
Changed lines of the file:
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@@
 </autorouter>
 <elements>
-<element name="C1" library="rcl" package="E2,5-5" value="100uF" x="7.62" y="3.81" rot="R270"/>
-<element name="C2" library="rcl" package="E2,5-5" value="22uF" x="22.86" y="3.81" rot="R270"/>
+<element name="C1" library="rcl" package="E2,5-5" value="100μF" x="7.62" y="3.81" rot="R270"/>
+<element name="C2" library="rcl" package="E2,5-5" value="22μF" x="22.86" y="3.81" rot="R270"/>
 <element name="D1" library="JDM2" package="DO35-5" value="1N4148" x="2.54" y="5.08" rot="R270"/>
 <element name="D2" library="JDM2" package="DO35Z5" value="Z=8.1V" x="20.32" y="10.16"/>
@@
 <element name="LED1" library="1dmf" package="LED5MM" value="Power" x="38.1" y="3.81" rot="R270"/>
 <element name="LED2" library="1dmf" package="LED5MM" value="Vpp" x="15.24" y="3.81" rot="R270"/>
-<element name="R1" library="JDM2" package="0207/10" value="10k" x="33.02" y="22.86" rot="R180"/>
-<element name="R2" library="JDM2" package="0204/7" value="1.5k" x="40.64" y="16.51" rot="R90"/>
-<element name="R4" library="JDM2" package="0207/10" value="1K" x="7.62" y="25.4" rot="R180"/>
-<element name="R5" library="JDM2" package="0207/10" value="15K" x="7.62" y="27.94" rot="R180"/>
-<element name="R6" library="JDM2" package="0207/10" value="4.7k" x="12.7" y="10.16" rot="R90"/>
-<element name="R7" library="JDM2" package="0207/10" value="1k" x="35.56" y="10.16" rot="R90"/>
+<element name="R1" library="JDM2" package="0207/10" value="10kΩ" x="33.02" y="22.86" rot="R180"/>
+<element name="R2" library="JDM2" package="0204/7" value="1.5kΩ" x="40.64" y="16.51" rot="R90"/>
+<element name="R4" library="JDM2" package="0207/10" value="1kΩ" x="7.62" y="25.4" rot="R180"/>
+<element name="R5" library="JDM2" package="0207/10" value="15kΩ" x="7.62" y="27.94" rot="R180"/>
+<element name="R6" library="JDM2" package="0207/10" value="4.7kΩ" x="12.7" y="10.16" rot="R90"/>
+<element name="R7" library="JDM2" package="0207/10" value="1kΩ" x="35.56" y="10.16" rot="R90"/>
 <element name="T1" library="JDM2" package="TO92-CBE" value="BC547" x="7.62" y="12.7" rot="R90"/>
 <element name="T2" library="JDM2" package="TO92-CBE" value="BC547" x="43.18" y="25.4" rot="R90"/>

Commit message: ...
Changed lines of the file:
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@@
 <description>JDM2 without DIL-Socket</description>
 <plain>
-<wire x1="0" y1="0" x2="48.24" y2="0" width="0" layer="47"/>
-<wire x1="48.24" y1="0" x2="48.26" y2="30.48" width="0" layer="47"/>
-<wire x1="48.26" y1="30.48" x2="0" y2="30.48" width="0" layer="47"/>
-<wire x1="0" y1="30.48" x2="0" y2="0" width="0" layer="47"/>
+<wire x1="0" y1="0" x2="48.24" y2="0" width="0" layer="20"/>
+<wire x1="48.24" y1="0" x2="48.26" y2="30.48" width="0" layer="20"/>
+<wire x1="48.26" y1="30.48" x2="0" y2="30.48" width="0" layer="20"/>
+<wire x1="0" y1="30.48" x2="0" y2="0" width="0" layer="20"/>
 </plain>
 <attributes>
