File: eagle/JDM2_NoSocket.Old.brd (EAGLE design)
At the start: 18 parts, among them Q2 BC547, T2 BC547

Commit message: ...
Parts:
- R1: value 10k -> 10kΩ
- R2: value 1k5 -> 1.5kΩ
- R4: value 1K -> 1kΩ
- R5: value 15K -> 15kΩ
Changed lines of the file:
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@@
 <element name="RS232" library="pinhead" package="1X05" value="" x="48.26" y="48.26" rot="R90"/>
 <element name="Q2" library="JDM2" package="TO92-CBE" value="BC547" x="43.18" y="55.88" rot="R90"/>
-<element name="R1" library="rcl" package="0204/7" value="10k" x="40.64" y="52.07" rot="R270"/>
-<element name="R2" library="rcl" package="0207/7" value="1k5" x="45.72" y="49.53" rot="R90"/>
-<element name="R4" library="rcl" package="0204/7" value="1K" x="22.86" y="44.45" rot="R90"/>
-<element name="R5" library="rcl" package="0204/5" value="15K" x="27.94" y="45.72" rot="R90"/>
+<element name="R1" library="rcl" package="0204/7" value="10kΩ" x="40.64" y="52.07" rot="R270"/>
+<element name="R2" library="rcl" package="0207/7" value="1.5kΩ" x="45.72" y="49.53" rot="R90"/>
+<element name="R4" library="rcl" package="0204/7" value="1kΩ" x="22.86" y="44.45" rot="R90"/>
+<element name="R5" library="rcl" package="0204/5" value="15kΩ" x="27.94" y="45.72" rot="R90"/>
 <element name="SV3" library="con-lstb" package="MA03-1" value="" x="17.78" y="40.64">
 <attribute name="MF" value="" x="17.78" y="40.64" size="1.778" layer="27" display="off"/>

Commit message: ...
Other:
- board outline added: 160 x 100 mm
Changed lines of the file:
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@@
 <description>JDM2 without DIL-Socket</description>
 <plain>
-<wire x1="0" y1="0" x2="160" y2="0" width="0" layer="47"/>
-<wire x1="160" y1="0" x2="160" y2="100" width="0" layer="47"/>
-<wire x1="160" y1="100" x2="0" y2="100" width="0" layer="47"/>
-<wire x1="0" y1="100" x2="0" y2="0" width="0" layer="47"/>
+<wire x1="0" y1="0" x2="160" y2="0" width="0" layer="20"/>
+<wire x1="160" y1="0" x2="160" y2="100" width="0" layer="20"/>
+<wire x1="160" y1="100" x2="0" y2="100" width="0" layer="20"/>
+<wire x1="0" y1="100" x2="0" y2="0" width="0" layer="20"/>
 </plain>
 <attributes>
