File: eagle/JDM2_NoSocket_Mirrored.brd (EAGLE design)
At the start: 17 parts, among them J1 COMPORT-6PIN, T1 BC547CBE-A, T2 BC547CBE

Commit message: ...
Parts:
- C1: value 100uF -> 100μF
- C2: value 22uF -> 22μF
- R1: value 10k -> 10kΩ
- R2: value 1.5k -> 1.5kΩ
- R3: value 100 -> 100Ω
Changed lines of the file:
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@@
 </autorouter>
 <elements>
-<element name="C1" library="c" package="E5-4" value="100uF" x="63.5" y="20.32" rot="R90"/>
-<element name="C2" library="c" package="E2,5-4" value="22uF" x="52.07" y="17.78" rot="R180"/>
+<element name="C1" library="c" package="E5-4" value="100μF" x="63.5" y="20.32" rot="R90"/>
+<element name="C2" library="c" package="E2,5-4" value="22μF" x="52.07" y="17.78" rot="R180"/>
 <element name="D1" library="d" package="DO34-2,5-A" value="1N4148" x="71.12" y="16.51" rot="R90"/>
 <element name="D4" library="d" package="DO34Z5" value="Z=8.1V" x="58.42" y="22.86" smashed="yes" rot="R90">
@@
 <attribute name="VALUE" x="60.325" y="27.051" size="1.27" layer="27" ratio="10" rot="R180"/>
 </element>
-<element name="R1" library="r" package="0202/5" value="10k" x="50.8" y="22.86" rot="R180"/>
-<element name="R2" library="r" package="0202/7" value="1.5k" x="48.26" y="21.59"/>
+<element name="R1" library="r" package="0202/5" value="10kΩ" x="50.8" y="22.86" rot="R180"/>
+<element name="R2" library="r" package="0202/7" value="1.5kΩ" x="48.26" y="21.59"/>
 <element name="T1" library="t" package="TO92-CBE-A" value="BC547CBE-A" x="68.58" y="22.86" rot="R90"/>
 <element name="T2" library="t" package="TO92-CBE" value="BC547CBE" x="50.8" y="27.94" rot="R90"/>
-<element name="R3" library="r" package="0202/5" value="100" x="55.88" y="30.48" rot="R90"/>
+<element name="R3" library="r" package="0202/5" value="100Ω" x="55.88" y="30.48" rot="R90"/>
 <element name="U$5" library="pinconn" package="PIC-ICSP" value="PIC-ICSPICSP" x="76.2" y="22.86" rot="R90"/>
 <element name="U$7" library="sw" package="SLSW-2P2T-H" value="SL-SW-2P-2T-H" x="16.51" y="38.1"/>

Commit message: ...
Other:
- board outline added: 166.3 x 87.3 mm
Changed lines of the file:
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@@
 <description>JDM2 without DIL-Socket</description>
 <plain>
-<wire x1="6.35" y1="12.7" x2="166.35" y2="12.7" width="0" layer="47"/>
-<wire x1="166.35" y1="12.7" x2="160" y2="100" width="0" layer="47"/>
-<wire x1="160" y1="100" x2="0" y2="100" width="0" layer="47"/>
-<wire x1="0" y1="100" x2="6.35" y2="12.7" width="0" layer="47"/>
+<wire x1="6.35" y1="12.7" x2="166.35" y2="12.7" width="0" layer="20"/>
+<wire x1="166.35" y1="12.7" x2="160" y2="100" width="0" layer="20"/>
+<wire x1="160" y1="100" x2="0" y2="100" width="0" layer="20"/>
+<wire x1="0" y1="100" x2="6.35" y2="12.7" width="0" layer="20"/>
 </plain>
 <attributes>
