File: eagle/RS232_2xNPN.brd (EAGLE design)
At the start: 9 parts, among them J1 COMPORT-4PIN-NEW, J2 PIC-UART-X, T1 BC547, T2 BC547

Commit message: ...
Parts:
- R1: value 4.7k -> 4.7kΩ
- R4: value 10k -> 10kΩ
- R5, R6: value 1k -> 1kΩ
Changed lines of the file:
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@@
 <attribute name="VALUE" x="19.558" y="3.84175" size="0.4064" layer="27" ratio="10" align="top-center"/>
 </element>
-<element name="R1" library="r" package="0202/7" value="4.7k" x="19.05" y="5.08" smashed="yes">
+<element name="R1" library="r" package="0202/7" value="4.7kΩ" x="19.05" y="5.08" smashed="yes">
 <attribute name="NAME" x="21.336" y="4.191" size="0.6096" layer="25" ratio="10" align="top-center"/>
 <attribute name="VALUE" x="19.05" y="5.08" size="0.6096" layer="27" ratio="10" align="center"/>
 </element>
-<element name="R4" library="r" package="0202/7-V" value="10k" x="7.62" y="6.35"/>
-<element name="R5" library="r" package="0202/7-V" value="1k" x="5.08" y="8.89"/>
+<element name="R4" library="r" package="0202/7-V" value="10kΩ" x="7.62" y="6.35"/>
+<element name="R5" library="r" package="0202/7-V" value="1kΩ" x="5.08" y="8.89"/>
 <element name="T1" library="t" package="TO92-CBE" value="BC547" x="20.32" y="10.16" smashed="yes">
 <attribute name="NAME" x="21.336" y="8.89" size="0.8128" layer="25" ratio="10" align="center"/>
@@
 <attribute name="VALUE" x="11.684" y="6.4135" size="0.6096" layer="27" ratio="10" align="center"/>
 </element>
-<element name="R6" library="r" package="0202/7" value="1k" x="13.97" y="12.7" rot="R180"/>
+<element name="R6" library="r" package="0202/7" value="1kΩ" x="13.97" y="12.7" rot="R180"/>
 <element name="J2" library="pinconn" package="PIC-UART-X" value="PIC-UART-X" x="2.54" y="6.35" smashed="yes">
 <attribute name="NAME" x="3.048" y="11.938" size="0.8128" layer="25" rot="R180" align="top-left"/>

Commit message: ...
Other:
- board outline added: 27.9 x 15.2 mm
Changed lines of the file:
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@@
 <description>RS232 Adapter using two NPN Transistors</description>
 <plain>
-<wire x1="27.94" y1="15.24" x2="0.02" y2="15.24" width="0.127" layer="47"/>
-<wire x1="0.02" y1="15.24" x2="0.02" y2="0" width="0.127" layer="47"/>
-<wire x1="0.02" y1="0" x2="27.94" y2="0" width="0.127" layer="47"/>
-<wire x1="27.94" y1="0" x2="27.94" y2="15.24" width="0.127" layer="47"/>
+<wire x1="27.94" y1="15.24" x2="0.02" y2="15.24" width="0.127" layer="20"/>
+<wire x1="0.02" y1="15.24" x2="0.02" y2="0" width="0.127" layer="20"/>
+<wire x1="0.02" y1="0" x2="27.94" y2="0" width="0.127" layer="20"/>
+<wire x1="27.94" y1="0" x2="27.94" y2="15.24" width="0.127" layer="20"/>
 </plain>
 <attributes>
