File: eagle/RS232_HCPL2730.brd (EAGLE design)
At the start: 7 parts

Commit message: ...
Routing:
- net GND: track 51.0 -> 50.0 mm
- net N$2: track 10.7 -> 10.1 mm
- net N$5: track 47.3 -> 46.8 mm

Commit message: ...
Parts:
- R1, R2: value 330 -> 330Ω
- R3, R4: value 4.7k -> 4.7kΩ
Changed lines of the file:
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@@
           <attribute name="MPN" value="HCPL-2730-000E" x="16.51" y="8.89" size="1.778" layer="27" rot="R270" display="off" />
         </element>
-        <element name="R1" library="resistor" package="0207/10" value="330" x="7.62" y="7.62" rot="R90" />
-        <element name="R2" library="resistor" package="0204/7" value="330" x="35.56" y="6.35" rot="R90" />
-        <element name="R3" library="resistor" package="0204/7" value="4.7k" x="29.21" y="7.62" />
-        <element name="R4" library="resistor" package="0204/7" value="4.7k" x="29.21" y="12.7" />
+        <element name="R1" library="resistor" package="0207/10" value="330Ω" x="7.62" y="7.62" rot="R90" />
+        <element name="R2" library="resistor" package="0204/7" value="330Ω" x="35.56" y="6.35" rot="R90" />
+        <element name="R3" library="resistor" package="0204/7" value="4.7kΩ" x="29.21" y="7.62" />
+        <element name="R4" library="resistor" package="0204/7" value="4.7kΩ" x="29.21" y="12.7" />
         <element name="U$2" library="pinconn" package="CONN-6P" value="FTDI232-BO-6P" x="40.64" y="8.89" rot="R270" />
         <element name="U$3" library="pinconn" package="CONN-4P" value="PIC-UART-NOVDD-4P" x="2.54" y="7.62" rot="R270" />

Commit message: ...
Other:
- board outline added: 43.2 x 17.8 mm
Changed lines of the file:
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@@
 Powered by PIC</description>
       <plain>
-        <wire x1="0" y1="0" x2="43.18" y2="0" width="0" layer="47" />
-        <wire x1="43.18" y1="0" x2="43.18" y2="17.78" width="0" layer="47" />
-        <wire x1="43.18" y1="17.78" x2="0" y2="17.78" width="0" layer="47" />
-        <wire x1="0" y1="17.78" x2="0" y2="0" width="0" layer="47" />
+        <wire x1="0" y1="0" x2="43.18" y2="0" width="0" layer="20" />
+        <wire x1="43.18" y1="0" x2="43.18" y2="17.78" width="0" layer="20" />
+        <wire x1="43.18" y1="17.78" x2="0" y2="17.78" width="0" layer="20" />
+        <wire x1="0" y1="17.78" x2="0" y2="0" width="0" layer="20" />
       </plain>
       <attributes></attributes>
