File: eagle/RS232_NPN_PNP.brd (EAGLE design)
At the start: 10 parts, among them J1 FTDI232, J2 PIC-UART, T1 BC547, T2 BC557

Commit message: ...
Parts:
- R1, R4: value 10k -> 10kΩ
- R2, R5: value 1k -> 1kΩ
- R3: value 4.7k -> 4.7kΩ
Changed lines of the file:
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@@
 <elements>
 <element name="D1" library="d" package="DO34-5" value="1N4148" x="17.78" y="10.16"/>
-<element name="R1" library="r" package="0202/5-V" value="10k" x="5.08" y="7.62"/>
-<element name="R2" library="r" package="0202/5-V" value="1k" x="7.62" y="5.08"/>
-<element name="R3" library="r" package="0202/5-V" value="4.7k" x="10.16" y="10.16"/>
-<element name="R4" library="r" package="0202/5" value="10k" x="15.24" y="5.08" rot="R180"/>
-<element name="R5" library="r" package="0202/5-V" value="1k" x="20.32" y="5.08"/>
+<element name="R1" library="r" package="0202/5-V" value="10kΩ" x="5.08" y="7.62"/>
+<element name="R2" library="r" package="0202/5-V" value="1kΩ" x="7.62" y="5.08"/>
+<element name="R3" library="r" package="0202/5-V" value="4.7kΩ" x="10.16" y="10.16"/>
+<element name="R4" library="r" package="0202/5" value="10kΩ" x="15.24" y="5.08" rot="R180"/>
+<element name="R5" library="r" package="0202/5-V" value="1kΩ" x="20.32" y="5.08"/>
 <element name="T2" library="t" package="TO92-CBE" value="BC557" x="12.7" y="2.54" smashed="yes" rot="R90">
 <attribute name="NAME" x="11.684" y="3.81" size="0.8128" layer="25" ratio="10" rot="R180" align="center"/>

Commit message: ...
Other:
- board outline added: 27.9 x 15.2 mm
Changed lines of the file:
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@@
 <description>RS232 Adapter using NPN and PNP Transistors</description>
 <plain>
-<wire x1="0" y1="0" x2="27.92" y2="0" width="0" layer="47"/>
-<wire x1="27.92" y1="0" x2="27.94" y2="15.24" width="0" layer="47"/>
-<wire x1="27.94" y1="15.24" x2="0" y2="15.24" width="0" layer="47"/>
-<wire x1="0" y1="15.24" x2="0" y2="0" width="0" layer="47"/>
+<wire x1="0" y1="0" x2="27.92" y2="0" width="0" layer="20"/>
+<wire x1="27.92" y1="0" x2="27.94" y2="15.24" width="0" layer="20"/>
+<wire x1="27.94" y1="15.24" x2="0" y2="15.24" width="0" layer="20"/>
+<wire x1="0" y1="15.24" x2="0" y2="0" width="0" layer="20"/>
 </plain>
 <attributes>
