File: eagle/RS232_NPN_PNP_FTDI_2.brd (EAGLE design)
At the start: 11 parts, among them J1 FTDI232-BO-5P-L, J2 PIC-UART, T1 BC557, T2 BC547

Commit message: ...
Parts:
- C1: value 10uF -> 10μF
- R1, R2, R3, R4, R5: value 10k -> 10kΩ
Changed lines of the file:
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@@
 <elements>
 <element name="D1" library="d" package="DO34-5V" value="1N4148" x="7.62" y="7.62"/>
-<element name="R1" library="r" package="0202/7-V" value="10k" x="5.08" y="6.35"/>
-<element name="R2" library="r" package="0202/5" value="10k" x="17.78" y="5.08" rot="R180"/>
-<element name="R3" library="r" package="0202/5" value="10k" x="17.78" y="7.62" rot="R180"/>
-<element name="R4" library="r" package="0202/5" value="10k" x="17.78" y="10.16" rot="R180"/>
-<element name="R5" library="r" package="0202/5" value="10k" x="27.94" y="10.16" rot="R180"/>
+<element name="R1" library="r" package="0202/7-V" value="10kΩ" x="5.08" y="6.35"/>
+<element name="R2" library="r" package="0202/5" value="10kΩ" x="17.78" y="5.08" rot="R180"/>
+<element name="R3" library="r" package="0202/5" value="10kΩ" x="17.78" y="7.62" rot="R180"/>
+<element name="R4" library="r" package="0202/5" value="10kΩ" x="17.78" y="10.16" rot="R180"/>
+<element name="R5" library="r" package="0202/5" value="10kΩ" x="27.94" y="10.16" rot="R180"/>
 <element name="T1" library="t" package="TO92-CBE" value="BC557" x="15.24" y="2.54" smashed="yes" rot="R90">
 <attribute name="NAME" x="14.224" y="3.81" size="0.8128" layer="25" ratio="10" rot="R180" align="center"/>
@@
 <attribute name="VALUE" x="22.86" y="8.89" size="0.6096" layer="27" ratio="10" align="center"/>
 </element>
-<element name="C1" library="c" package="E2.5-4/V" value="10uF" x="10.16" y="10.16"/>
+<element name="C1" library="c" package="E2.5-4/V" value="10μF" x="10.16" y="10.16"/>
 <element name="J2" library="pinconn" package="PIC-UART" value="PIC-UART" x="33.02" y="5.08" smashed="yes">
 <attribute name="NAME" x="34.036" y="3.175" size="0.8128" layer="25" align="top-right"/>

Commit message: ...
Other:
- board outline added: 34.3 x 15.2 mm
Changed lines of the file:
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@@
 <description>RS232 Adapter using NPN and PNP Transistors</description>
 <plain>
-<wire x1="0" y1="15.24" x2="34.29" y2="15.24" width="0" layer="47"/>
-<wire x1="34.29" y1="15.24" x2="34.29" y2="0" width="0" layer="47"/>
-<wire x1="34.29" y1="0" x2="0" y2="0" width="0" layer="47"/>
-<wire x1="0" y1="0" x2="0" y2="15.24" width="0" layer="47"/>
+<wire x1="0" y1="15.24" x2="34.29" y2="15.24" width="0" layer="20"/>
+<wire x1="34.29" y1="15.24" x2="34.29" y2="0" width="0" layer="20"/>
+<wire x1="34.29" y1="0" x2="0" y2="0" width="0" layer="20"/>
+<wire x1="0" y1="0" x2="0" y2="15.24" width="0" layer="20"/>
 </plain>
 <attributes>
