File: eagle/RS232_NPN_PNP_Negative_Mirrored.brd (EAGLE design)
At the start: 11 parts, among them J1 COMPORT-4PIN-NEW, J2 PIC UART (4pin), T1 BC557, T2 BC547

Commit message: ...
Parts:
- C1: value 10uF -> 10μF
- R1, R2, R3, R4, R5: value 10k -> 10kΩ
Changed lines of the file:
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@@
 <elements>
 <element name="D1" library="d" package="DO34-7" value="1N4148" x="-15.24" y="8.89" rot="R180"/>
-<element name="R1" library="r" package="0202/7" value="10k" x="-15.24" y="11.43"/>
-<element name="R2" library="r" package="0202/10-V" value="10k" x="-26.67" y="6.35"/>
-<element name="R3" library="r" package="0202/7-V" value="10k" x="-24.13" y="5.08"/>
-<element name="R4" library="r" package="0202/7" value="10k" x="-15.24" y="3.81"/>
-<element name="R5" library="r" package="0202/7" value="10k" x="-15.24" y="1.27"/>
+<element name="R1" library="r" package="0202/7" value="10kΩ" x="-15.24" y="11.43"/>
+<element name="R2" library="r" package="0202/10-V" value="10kΩ" x="-26.67" y="6.35"/>
+<element name="R3" library="r" package="0202/7-V" value="10kΩ" x="-24.13" y="5.08"/>
+<element name="R4" library="r" package="0202/7" value="10kΩ" x="-15.24" y="3.81"/>
+<element name="R5" library="r" package="0202/7" value="10kΩ" x="-15.24" y="1.27"/>
 <element name="T1" library="t" package="TO92-CBE" value="BC557" x="-21.59" y="11.43" smashed="yes">
 <attribute name="NAME" x="-20.574" y="10.16" size="0.6096" layer="25" ratio="10" align="center"/>
@@
 </element>
 <element name="T2" library="t" package="TO92-CBE" value="BC547" x="-21.59" y="3.81" rot="R180"/>
-<element name="C1" library="c" package="E2,5-3" value="10uF" x="-15.24" y="6.35" smashed="yes" rot="R180">
+<element name="C1" library="c" package="E2,5-3" value="10μF" x="-15.24" y="6.35" smashed="yes" rot="R180">
 <attribute name="NAME" x="-13.462" y="5.5245" size="0.8128" layer="25" rot="R180" align="bottom-right"/>
 <attribute name="VALUE" x="-16.764" y="7.874" size="0.6096" layer="27" rot="R180"/>

Commit message: ...
Other:
- board outline added: 25.4 x 15.2 mm
Changed lines of the file:
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@@
 <description>RS232 Adapter using NPN and PNP Transistors</description>
 <plain>
-<wire x1="-31.75" y1="15.24" x2="-6.35" y2="15.24" width="0" layer="47"/>
-<wire x1="-6.35" y1="15.24" x2="-6.35" y2="0" width="0" layer="47"/>
-<wire x1="-6.35" y1="0" x2="-31.75" y2="0" width="0" layer="47"/>
-<wire x1="-31.75" y1="0" x2="-31.75" y2="15.24" width="0" layer="47"/>
+<wire x1="-31.75" y1="15.24" x2="-6.35" y2="15.24" width="0" layer="20"/>
+<wire x1="-6.35" y1="15.24" x2="-6.35" y2="0" width="0" layer="20"/>
+<wire x1="-6.35" y1="0" x2="-31.75" y2="0" width="0" layer="20"/>
+<wire x1="-31.75" y1="0" x2="-31.75" y2="15.24" width="0" layer="20"/>
 </plain>
 <attributes>
