File: eagle/TTL_Inverter.brd (EAGLE design)
At the start: 9 parts

Commit message: ...
Parts:
- R1: value 1k -> 1kΩ
- R2, R3: value 10k -> 10kΩ
- R4: value 15k -> 15kΩ
- R5: value 4.7k -> 4.7kΩ
Changed lines of the file:
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@@
 </autorouter>
 <elements>
-<element name="R1" library="resistor" package="0207/2V" value="1k" x="43.18" y="29.21" rot="R270"/>
-<element name="R2" library="resistor" package="0207/7" value="10k" x="35.56" y="21.59" rot="R270"/>
-<element name="R3" library="resistor" package="0207/10" value="10k" x="48.26" y="25.4" rot="R270"/>
-<element name="R4" library="resistor" package="0207/10" value="15k" x="45.72" y="25.4" rot="R270"/>
-<element name="R5" library="resistor" package="0207/2V" value="4.7k" x="41.91" y="17.78"/>
+<element name="R1" library="resistor" package="0207/2V" value="1kΩ" x="43.18" y="29.21" rot="R270"/>
+<element name="R2" library="resistor" package="0207/7" value="10kΩ" x="35.56" y="21.59" rot="R270"/>
+<element name="R3" library="resistor" package="0207/10" value="10kΩ" x="48.26" y="25.4" rot="R270"/>
+<element name="R4" library="resistor" package="0207/10" value="15kΩ" x="45.72" y="25.4" rot="R270"/>
+<element name="R5" library="resistor" package="0207/2V" value="4.7kΩ" x="41.91" y="17.78"/>
 <element name="T1" library="transistor" package="TO92-CBE" value="" x="40.64" y="25.4" rot="R270"/>
 <element name="T2" library="transistor" package="TO92-CBE" value="" x="48.26" y="17.78"/>

Commit message: ...
Other:
- board outline added: 100 x 80 mm
Changed lines of the file:
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@@
 <board>
 <plain>
-<wire x1="0" y1="0" x2="100" y2="0" width="0" layer="47"/>
-<wire x1="100" y1="0" x2="100" y2="80" width="0" layer="47"/>
-<wire x1="100" y1="80" x2="0" y2="80" width="0" layer="47"/>
-<wire x1="0" y1="80" x2="0" y2="0" width="0" layer="47"/>
+<wire x1="0" y1="0" x2="100" y2="0" width="0" layer="20"/>
+<wire x1="100" y1="0" x2="100" y2="80" width="0" layer="20"/>
+<wire x1="100" y1="80" x2="0" y2="80" width="0" layer="20"/>
+<wire x1="0" y1="80" x2="0" y2="0" width="0" layer="20"/>
 <text x="57.15" y="27.94" size="1.016" layer="16" align="center-left">RxD</text>
 <text x="57.15" y="30.48" size="1.016" layer="16" align="center-left">TxD</text>
