File: eagle/Urzeitcode - 18F16Q41.sch (EAGLE design)
At the start: 9 parts, among them IC1 PIC18F16Q41-I/P, IC2 MCP3301, J1 PICKIT3-ICSP-ICSP, SW1 PB-1P-1T2P1T, SW2 PB-1P-1T2P1T

Commit message: ...
Connections:
- net N$1 renamed RC5
- net N$2 renamed RC4
- net N$3 renamed RC3
- net N$4 renamed RC6
- net N$5 renamed RC7
- net N$7 renamed RB7
Changed lines of the file:
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@@
 </segment>
 </net>
-<net name="N$1" class="0">
+<net name="RC5" class="0">
 <segment>
 <pinref part="IC1" gate="G$1" pin="RC5"/>
@@
 </segment>
 </net>
-<net name="N$2" class="0">
+<net name="RC4" class="0">
 <segment>
 <pinref part="U$2" gate="G$1" pin="SDIN"/>
@@
 </segment>
 </net>
-<net name="N$3" class="0">
+<net name="RC3" class="0">
 <segment>
 <pinref part="U$2" gate="G$1" pin="D_C"/>
@@
 </segment>
 </net>
-<net name="N$4" class="0">
+<net name="RC6" class="0">
 <segment>
 <pinref part="U$2" gate="G$1" pin="RES"/>
@@
 </segment>
 </net>
-<net name="N$5" class="0">
+<net name="RC7" class="0">
 <segment>
 <pinref part="U$2" gate="G$1" pin="SCE"/>
@@
 </segment>
 </net>
-<net name="N$7" class="0">
+<net name="RB7" class="0">
 <segment>
 <pinref part="R1" gate="1" pin="2"/>
