File: eagle/OpenProg-18F2550.brd (EAGLE design)
At the start: 137.2 x 78.7 mm, 45 parts, among them J1 CONN-10P, J3 USB-SH, T1 BC557, T2 BC557, T3 BC547, T4 BC547, U1 PIC18F2550-I/SP-V, X1 12MHz

Commit message: ...
Parts:
- C1: value 100uF -> 100μF
- C6: value 10uF -> 10μF
- R1: value 22k -> 22kΩ
- R10, R11, R12, R13, R3, R5, R6: value 100k -> 100kΩ
- R14, R15, R16, R17, R18, R19, R20, R21, R22, R23: value 100 -> 100Ω
- R2: value 12k -> 12kΩ
- R24, R25: value 330k -> 330kΩ
- R7: value 1M -> 1MΩ
- R8, R9: value 2.2k -> 2.2kΩ
Changed lines of the file:
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@@
       </autorouter>
       <elements>
-        <element name="C1" library="c" package="E5-5" value="100uF" x="55.88" y="15.24" rot="R90" />
+        <element name="C1" library="c" package="E5-5" value="100μF" x="55.88" y="15.24" rot="R90" />
         <element name="C2" library="c" package="C025-020X036" value="22pF" x="72.39" y="38.1" />
         <element name="C3" library="c" package="C025-020X036" value="22pF" x="72.39" y="33.02" />
         <element name="C4" library="c" package="C050-030X075" value="330nF" x="78.74" y="20.32" rot="R270" />
         <element name="C5" library="c" package="C050-025X075" value="100nF" x="40.64" y="25.4" />
-        <element name="C6" library="c" package="E5-5" value="10uF" x="104.14" y="15.24" rot="R270" />
+        <element name="C6" library="c" package="E5-5" value="10μF" x="104.14" y="15.24" rot="R270" />
         <element name="C7" library="c" package="C050-025X075" value="100nF" x="45.72" y="35.56" />
         <element name="C8" library="c" package="C050-025X075" value="100nF" x="66.04" y="12.7" rot="R180" />
@@
         <element name="J3" library="usb" package="USB-B-PRINT" value="USB-SH" x="91.44" y="11.43" />
         <element name="L1" library="l" package="L-03/10V" value="" x="58.42" y="25.4" rot="R90" />
-        <element name="R1" library="r" package="0204/10-V" value="22k" x="43.18" y="15.24" />
-        <element name="R10" library="r" package="0204/10" value="100k" x="76.2" y="25.4" />
-        <element name="R18" library="r" package="0204/10" value="100" x="101.6" y="45.72" />
-        <element name="R14" library="r" package="0204/10" value="100" x="101.6" y="55.88" />
-        <element name="R15" library="r" package="0204/10" value="100" x="101.6" y="53.34" />
-        <element name="R17" library="r" package="0204/10" value="100" x="101.6" y="48.26" />
-        <element name="R19" library="r" package="0204/10" value="100" x="101.6" y="43.18" />
-        <element name="R2" library="r" package="0204/10-V" value="12k" x="50.8" y="20.32" rot="R270" />
-        <element name="R20" library="r" package="0204/10" value="100" x="101.6" y="40.64" />
-        <element name="R21" library="r" package="0204/10" value="100" x="101.6" y="38.1" />
-        <element name="R22" library="r" package="0204/10" value="100" x="101.6" y="30.48" />
-        <element name="R23" library="r" package="0204/10" value="100" x="101.6" y="27.94" />
-        <element name="R24" library="r" package="0204/10-V" value="330k" x="43.18" y="38.1" rot="R90" />
-        <element name="R25" library="r" package="0204/10-V" value="330k" x="43.18" y="33.02" rot="R90" />
-        <element name="R3" library="r" package="0204/10" value="100k" x="60.96" y="43.18" rot="R180" />
-        <element name="R5" library="r" package="0204/10" value="100k" x="76.2" y="27.94" />
-        <element name="R6" library="r" package="0204/10" value="100k" x="76.2" y="30.48" />
-        <element name="R16" library="r" package="0204/10" value="100" x="101.6" y="50.8" />
+        <element name="R1" library="r" package="0204/10-V" value="22kΩ" x="43.18" y="15.24" />
+        <element name="R10" library="r" package="0204/10" value="100kΩ" x="76.2" y="25.4" />
+        <element name="R18" library="r" package="0204/10" value="100Ω" x="101.6" y="45.72" />
+        <element name="R14" library="r" package="0204/10" value="100Ω" x="101.6" y="55.88" />
+        <element name="R15" library="r" package="0204/10" value="100Ω" x="101.6" y="53.34" />
+        <element name="R17" library="r" package="0204/10" value="100Ω" x="101.6" y="48.26" />
+        <element name="R19" library="r" package="0204/10" value="100Ω" x="101.6" y="43.18" />
+        <element name="R2" library="r" package="0204/10-V" value="12kΩ" x="50.8" y="20.32" rot="R270" />
+        <element name="R20" library="r" package="0204/10" value="100Ω" x="101.6" y="40.64" />
+        <element name="R21" library="r" package="0204/10" value="100Ω" x="101.6" y="38.1" />
+        <element name="R22" library="r" package="0204/10" value="100Ω" x="101.6" y="30.48" />
+        <element name="R23" library="r" package="0204/10" value="100Ω" x="101.6" y="27.94" />
+        <element name="R24" library="r" package="0204/10-V" value="330kΩ" x="43.18" y="38.1" rot="R90" />
+        <element name="R25" library="r" package="0204/10-V" value="330kΩ" x="43.18" y="33.02" rot="R90" />
+        <element name="R3" library="r" package="0204/10" value="100kΩ" x="60.96" y="43.18" rot="R180" />
+        <element name="R5" library="r" package="0204/10" value="100kΩ" x="76.2" y="27.94" />
+        <element name="R6" library="r" package="0204/10" value="100kΩ" x="76.2" y="30.48" />
+        <element name="R16" library="r" package="0204/10" value="100Ω" x="101.6" y="50.8" />
         <element name="T1" library="t" package="TO92-CBE-A" value="BC557" x="63.5" y="38.1" rot="R90" />
         <element name="T2" library="t" package="TO92-CBE-A" value="BC557" x="48.26" y="27.94" />
@@
         <element name="U1" library="mcu" package="DIL28-3/V" value="PIC18F2550-I/SP-V" x="88.9" y="39.37" />
         <element name="X1" library="q" package="HC49" value="12MHz" x="78.74" y="35.56" />
-        <element name="R11" library="r" package="0204/10" value="100k" x="76.2" y="45.72" />
-        <element name="R12" library="r" package="0204/10" value="100k" x="76.2" y="43.18" />
-        <element name="R13" library="r" package="0204/10" value="100k" x="76.2" y="40.64" />
-        <element name="R9" library="r" package="0204/10" value="2.2k" x="76.2" y="48.26" />
-        <element name="R8" library="r" package="0204/10" value="2.2k" x="76.2" y="50.8" />
-        <element name="R7" library="r" package="0204/10" value="1M" x="76.2" y="55.88" />
+        <element name="R11" library="r" package="0204/10" value="100kΩ" x="76.2" y="45.72" />
+        <element name="R12" library="r" package="0204/10" value="100kΩ" x="76.2" y="43.18" />
+        <element name="R13" library="r" package="0204/10" value="100kΩ" x="76.2" y="40.64" />
+        <element name="R9" library="r" package="0204/10" value="2.2kΩ" x="76.2" y="48.26" />
+        <element name="R8" library="r" package="0204/10" value="2.2kΩ" x="76.2" y="50.8" />
+        <element name="R7" library="r" package="0204/10" value="1MΩ" x="76.2" y="55.88" />
         <element name="SW1" library="sw" package="PB-1P1T" value="" x="71.12" y="60.96" rot="R180" />
         <element name="D1" library="d" package="LED5MM" value="YELLOW" x="67.31" y="50.8" rot="R180" />

Commit message: ...
Parts:
- C2, C3: device c:C025-020X036 -> c:C025-015X024
- D1, D2: device d:LED5MM -> d:LED_3MM
Connections:
- net FB: now also R1.2, R2.1; no longer R1.1, R2.2
- net GND: now also R2.2, R24.2, R25.2, T3.3, T4.3; no longer R2.1, R24.1, R25.1, T3.E, T4.E
- net N$1: now also R1.1; no longer R1.2
- net N$11: now also T1.2, T3.1; no longer T1.B, T3.C
- net N$12: now also T2.2; no longer T2.B
- net N$2: now also T4.2; no longer T4.B
- net N$5: now also T4.1; no longer T4.C
- net N$7: now also T3.2; no longer T3.B
- net VCC: now also T2.3; no longer T2.E
- net VDDU: now also R25.1, T2.1; no longer R25.2, T2.C
- net VPP: now also T1.3; no longer T1.E
- net VPPU: now also R24.1, T1.1; no longer R24.2, T1.C

Commit message: ...
Parts:
- moved C1 35.6 mm to (20.3, 15.2)
- moved C2 35.6 mm to (36.8, 38.1)
- moved C3 35.6 mm to (36.8, 33.0)
- moved C5 35.6 mm to (5.08, 25.4)
- moved C6 35.6 mm to (68.6, 15.2)
- moved C7 35.6 mm to (10.2, 35.6)
- moved C8 35.6 mm to (30.5, 12.7)
- moved D1 35.6 mm to (31.8, 50.8)
- moved D2 35.6 mm to (25.4, 48.3)
- moved D3 35.6 mm to (27.9, 19.1)
- moved J1 35.6 mm to (78.7, 45.7)
- moved L1 35.6 mm to (22.9, 25.4)
- moved R1 35.6 mm to (7.62, 15.2)
- moved R10 35.6 mm to (40.6, 25.4)
- moved R11 35.6 mm to (40.6, 45.7)
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Other:
- board size 137.2 x 78.7 mm -> 101.6 x 78.7 mm

Commit message: ...
Parts:
- moved R5 15.2 mm to (25.4, 27.9)
- moved R24 10.2 mm to (17.8, 38.1), turned to 270 degrees
- moved C5 8.03 mm to (12.7, 22.9), turned to 180 degrees
- moved C7 8.03 mm to (17.8, 33.0), turned to 270 degrees
- moved C8 5.08 mm to (30.5, 17.8), turned to 270 degrees
- moved R1 5.08 mm to (12.7, 15.2), turned to 270 degrees
- moved C1 3.59 mm to (22.9, 17.8)
- moved R2 2.54 mm to (12.7, 20.3), turned to 90 degrees
- moved J3 2.54 mm to (58.4, 11.4)
- moved R25 2.54 mm to (7.62, 35.6), turned to 180 degrees
- moved T2 2.54 mm to (10.2, 27.9)
Connections:
- net N$10 renamed RC2
- net N$8 renamed RC0
- net N$9 renamed RC1
Routing:
- net GND: track 0.00 -> 153.7 mm
- net VCC: track 0.00 -> 143.5 mm
- net N$34: track 0.00 -> 16.5 mm
- net N$33: track 0.00 -> 12.7 mm
- net N$32: track 0.00 -> 12.7 mm
- net OSC1: track 0.00 -> 8.89 mm
- net N$35: track 0.00 -> 6.35 mm
- net N$21: track 0.00 -> 3.81 mm

Commit message: ...
Parts:
- L1: value (none) -> 100µH
Changed lines of the file:
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@@
 <element name="J1" library="pinconn" package="CONN-10P" value="CONN-10P" x="78.74" y="45.72" rot="R270"/>
 <element name="J3" library="usb" package="USB-B-PRINT" value="USB-SH" x="58.42" y="11.43"/>
-<element name="L1" library="l" package="L-03/10V" value="" x="22.86" y="25.4" rot="R90"/>
+<element name="L1" library="l" package="L-03/10V" value="100µH" x="22.86" y="25.4" rot="R90"/>
 <element name="R1" library="r" package="0204/10-V" value="22kΩ" x="12.7" y="15.24" rot="R270"/>
 <element name="R10" library="r" package="0204/10" value="100kΩ" x="40.64" y="25.4"/>

Commit message: ...
Parts:
- removed R11, R12, R13: 100kΩ, r:0204/10
- R3: device r:0204/10 -> r:0204/2
- moved SW1 21.7 mm to (15.2, 53.3), turned to 270 degrees
- moved R25 14.8 mm to (20.3, 43.2), turned to 90 degrees
- moved R7 13.0 mm to (53.3, 58.4), turned to 180 degrees
- moved R24 8.03 mm to (25.4, 40.6)
- moved C8 7.62 mm to (38.1, 17.8)
- moved R3 6.84 mm to (22.9, 36.8), turned to 90 degrees
- moved C5 5.68 mm to (17.8, 20.3)
- moved T2 5.68 mm to (15.2, 30.5)
- moved R2 3.59 mm to (15.2, 17.8)
- moved C6 2.54 mm to (68.6, 17.8)
- moved J3 2.54 mm to (58.4, 14.0)
- moved R1 2.54 mm to (15.2, 15.2)
- moved C1 2.54 mm to (25.4, 17.8)
- moved C7 2.54 mm to (17.8, 35.6), turned to 180 degrees
- moved D3 2.54 mm to (30.5, 19.1)
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Connections:
- removed net N$38: D1.K, D2.K, SW1.1
- removed net N$41: R7.1
- removed net RA3: R11.1
- removed net RA4: R12.1
- removed net RA5: R13.1
- net GND: now also D1.K, D2.K, SW1.1
- net N$3: no longer R11.2
- net N$4: no longer R12.2
- net N$6: no longer R13.2
- net VCC: now also R7.1
Routing:
- net FB: track 0.00 -> 76.2 mm
- net RC1: track 0.00 -> 20.3 mm
- net VCC: track 143.5 -> 162.6 mm
- net N$1: track 0.00 -> 17.8 mm
- net GND: track 153.7 -> 165.1 mm
- net N$11: track 0.00 -> 10.2 mm
- net OSC2: track 0.00 -> 10.2 mm
- net N$7: track 0.00 -> 7.62 mm
- net N$5: track 0.00 -> 7.62 mm
- net VDDU: track 0.00 -> 7.62 mm
- net N$36: track 0.00 -> 5.08 mm
- net OSC1: track 8.89 -> 12.7 mm
- net N$35: track 6.35 -> 2.54 mm
- net N$34: track 16.5 -> 12.7 mm
- net VPPU: track 0.00 -> 2.54 mm
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
Commit message: ...
Routing:
- net N$37: track 0.00 -> 35.6 mm
- net N$40: track 0.00 -> 7.62 mm
- net N$29: track 0.00 -> 7.62 mm
- net N$28: track 0.00 -> 7.62 mm
- net N$27: track 0.00 -> 7.62 mm
- net N$26: track 0.00 -> 7.62 mm
- net N$25: track 0.00 -> 7.62 mm
- net N$24: track 0.00 -> 7.62 mm
- net N$23: track 0.00 -> 7.62 mm
- net N$22: track 0.00 -> 7.62 mm
- net N$19: track 0.00 -> 6.35 mm
- net N$31: track 0.00 -> 5.08 mm
- net N$30: track 0.00 -> 5.08 mm
- net N$20: track 0.00 -> 5.08 mm
- net N$18: track 0.00 -> 5.08 mm
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Other:
- board size 101.6 x 78.7 mm -> 78.7 x 58.4 mm
Changed lines of the file:
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@@
 <board>
 <plain>
-<wire x1="0" y1="0" x2="101.6" y2="0" width="0" layer="20"/>
-<wire x1="101.6" y1="0" x2="101.6" y2="78.74" width="0" layer="20"/>
-<wire x1="101.6" y1="78.74" x2="0" y2="78.74" width="0" layer="20"/>
-<wire x1="0" y1="78.74" x2="0" y2="0" width="0" layer="20"/>
+<wire x1="5.08" y1="5.08" x2="83.82" y2="5.08" width="0" layer="20"/>
+<wire x1="83.82" y1="5.08" x2="83.82" y2="63.5" width="0" layer="20"/>
+<wire x1="83.82" y1="63.5" x2="5.08" y2="63.5" width="0" layer="20"/>
+<wire x1="5.08" y1="63.5" x2="5.08" y2="5.08" width="0" layer="20"/>
 </plain>
 <attributes>
@@
 <contactref element="R10" pad="2"/>
 <contactref element="U1" pad="13"/>
-<wire x1="45.72" y1="25.4" x2="48.26" y2="25.4" width="0" layer="19" extent="1-1"/>
+<wire x1="45.72" y1="25.4" x2="48.26" y2="25.4" width="0.8128" layer="16"/>
 </signal>
 <signal name="VCC">
@@
 <contactref element="R25" pad="1"/>
 <wire x1="15.24" y1="35.56" x2="15.24" y2="43.18" width="0.8128" layer="16"/>
-<wire x1="15.24" y1="35.56" x2="15.24" y2="33.02" width="0" layer="19" extent="1-1"/>
+<wire x1="15.24" y1="35.56" x2="15.24" y2="33.02" width="0.8128" layer="16"/>
 </signal>
 <signal name="N$11">
@@
 <contactref element="T1" pad="2"/>
 <contactref element="R3" pad="2"/>
-<wire x1="30.48" y1="33.02" x2="27.94" y2="33.02" width="0.8128" layer="16"/>
-<wire x1="27.94" y1="33.02" x2="27.94" y2="35.56" width="0.8128" layer="16"/>
+<wire x1="30.48" y1="33.02" x2="30.48" y2="35.56" width="0.8128" layer="16"/>
+<wire x1="30.48" y1="35.56" x2="27.94" y2="35.56" width="0.8128" layer="16"/>
 <wire x1="27.94" y1="35.56" x2="22.86" y2="35.56" width="0.8128" layer="16"/>
 </signal>
@@
 <contactref element="R5" pad="1"/>
 <contactref element="T2" pad="2"/>
-<wire x1="17.78" y1="27.94" x2="17.78" y2="30.48" width="0" layer="19" extent="1-1"/>
+<wire x1="17.78" y1="27.94" x2="17.78" y2="30.48" width="0.8128" layer="16"/>
 </signal>
 <signal name="N$13">
 <contactref element="U1" pad="28"/>
 <contactref element="R14" pad="1"/>
-<wire x1="55.88" y1="55.88" x2="60.96" y2="55.88" width="0" layer="19" extent="1-1"/>
+<wire x1="55.88" y1="55.88" x2="60.96" y2="55.88" width="0.8128" layer="16"/>
 </signal>
 <signal name="N$15">
 <contactref element="R15" pad="1"/>
 <contactref element="U1" pad="27"/>
-<wire x1="55.88" y1="53.34" x2="60.96" y2="53.34" width="0" layer="19" extent="1-1"/>
+<wire x1="60.96" y1="53.34" x2="55.88" y2="53.34" width="0.8128" layer="16"/>
 </signal>
 <signal name="N$16">
 <contactref element="U1" pad="26"/>
 <contactref element="R16" pad="1"/>
-<wire x1="55.88" y1="50.8" x2="60.96" y2="50.8" width="0" layer="19" extent="1-1"/>
+<wire x1="55.88" y1="50.8" x2="60.96" y2="50.8" width="0.8128" layer="16"/>
 </signal>
 <signal name="N$17">
 <contactref element="U1" pad="25"/>
 <contactref element="R17" pad="1"/>
-<wire x1="55.88" y1="48.26" x2="60.96" y2="48.26" width="0" layer="19" extent="1-1"/>
+<wire x1="60.96" y1="48.26" x2="55.88" y2="48.26" width="0.8128" layer="16"/>
 </signal>
 <signal name="N$18">
 <contactref element="U1" pad="24"/>
 <contactref element="R18" pad="1"/>
-<wire x1="55.88" y1="45.72" x2="60.96" y2="45.72" width="0" layer="19" extent="1-1"/>
+<wire x1="55.88" y1="45.72" x2="60.96" y2="45.72" width="0.8128" layer="16"/>
 </signal>
 <signal name="N$19">
 <contactref element="U1" pad="23"/>
 <contactref element="R19" pad="1"/>
-<wire x1="55.88" y1="43.18" x2="60.96" y2="43.18" width="0" layer="19" extent="1-1"/>
+<wire x1="60.96" y1="43.18" x2="55.88" y2="43.18" width="0.8128" layer="16"/>
+<wire x1="54.61" y1="43.18" x2="55.88" y2="43.18" width="0.8128" layer="16"/>
 </signal>
 <signal name="N$20">
 <contactref element="U1" pad="22"/>
 <contactref element="R20" pad="1"/>
-<wire x1="55.88" y1="40.64" x2="60.96" y2="40.64" width="0" layer="19" extent="1-1"/>
+<wire x1="55.88" y1="40.64" x2="60.96" y2="40.64" width="0.8128" layer="16"/>
 </signal>
 <signal name="N$21">
@@
 <contactref element="R14" pad="2"/>
 <contactref element="J1" pad="1"/>
-<wire x1="71.12" y1="55.88" x2="78.74" y2="55.88" width="0" layer="19" extent="1-1"/>
+<wire x1="71.12" y1="55.88" x2="78.74" y2="55.88" width="0.8128" layer="16"/>
+<wire x1="80.01" y1="55.88" x2="78.74" y2="55.88" width="0" layer="19" extent="1-16"/>
 </signal>
 <signal name="N$23">
 <contactref element="R15" pad="2"/>
 <contactref element="J1" pad="2"/>
-<wire x1="71.12" y1="53.34" x2="78.74" y2="53.34" width="0" layer="19" extent="1-1"/>
+<wire x1="78.74" y1="53.34" x2="71.12" y2="53.34" width="0.8128" layer="16"/>
 </signal>
 <signal name="N$24">
 <contactref element="R16" pad="2"/>
 <contactref element="J1" pad="3"/>
-<wire x1="71.12" y1="50.8" x2="78.74" y2="50.8" width="0" layer="19" extent="1-1"/>
+<wire x1="71.12" y1="50.8" x2="78.74" y2="50.8" width="0.8128" layer="16"/>
 </signal>
 <signal name="N$25">
 <contactref element="R17" pad="2"/>
 <contactref element="J1" pad="4"/>
-<wire x1="71.12" y1="48.26" x2="78.74" y2="48.26" width="0" layer="19" extent="1-1"/>
+<wire x1="78.74" y1="48.26" x2="71.12" y2="48.26" width="0.8128" layer="16"/>
 </signal>
 <signal name="N$26">
 <contactref element="R18" pad="2"/>
 <contactref element="J1" pad="5"/>
-<wire x1="71.12" y1="45.72" x2="78.74" y2="45.72" width="0" layer="19" extent="1-1"/>
+<wire x1="71.12" y1="45.72" x2="78.74" y2="45.72" width="0.8128" layer="16"/>
 </signal>
 <signal name="N$27">
 <contactref element="R19" pad="2"/>
 <contactref element="J1" pad="6"/>
-<wire x1="71.12" y1="43.18" x2="78.74" y2="43.18" width="0" layer="19" extent="1-1"/>
+<wire x1="71.12" y1="43.18" x2="78.74" y2="43.18" width="0.8128" layer="16"/>
 </signal>
 <signal name="N$28">
 <contactref element="R20" pad="2"/>
 <contactref element="J1" pad="7"/>
-<wire x1="71.12" y1="40.64" x2="78.74" y2="40.64" width="0" layer="19" extent="1-1"/>
+<wire x1="78.74" y1="40.64" x2="71.12" y2="40.64" width="0.8128" layer="16"/>
 </signal>
 <signal name="N$29">
 <contactref element="R21" pad="2"/>
 <contactref element="J1" pad="8"/>
-<wire x1="71.12" y1="38.1" x2="78.74" y2="38.1" width="0" layer="19" extent="1-1"/>
+<wire x1="71.12" y1="38.1" x2="78.74" y2="38.1" width="0.8128" layer="16"/>
 </signal>
 <signal name="N$30">
 <contactref element="U1" pad="18"/>
 <contactref element="R22" pad="1"/>
-<wire x1="55.88" y1="30.48" x2="60.96" y2="30.48" width="0" layer="19" extent="1-1"/>
+<wire x1="55.88" y1="30.48" x2="60.96" y2="30.48" width="0.8128" layer="16"/>
 </signal>
 <signal name="N$31">
 <contactref element="U1" pad="17"/>
 <contactref element="R23" pad="1"/>
-<wire x1="55.88" y1="27.94" x2="60.96" y2="27.94" width="0" layer="19" extent="1-1"/>
+<wire x1="60.96" y1="27.94" x2="55.88" y2="27.94" width="0.8128" layer="16"/>
 </signal>
 <signal name="N$32">
@@
 <contactref element="U1" pad="4"/>
 <contactref element="R9" pad="2"/>
-<wire x1="45.72" y1="48.26" x2="48.26" y2="48.26" width="0" layer="19" extent="1-1"/>
+<wire x1="48.26" y1="48.26" x2="45.72" y2="48.26" width="0.8128" layer="16"/>
 </signal>
 <signal name="RA1">
 <contactref element="U1" pad="3"/>
 <contactref element="R8" pad="2"/>
-<wire x1="45.72" y1="50.8" x2="48.26" y2="50.8" width="0" layer="19" extent="1-1"/>
+<wire x1="45.72" y1="50.8" x2="48.26" y2="50.8" width="0.8128" layer="16"/>
+<wire x1="49.53" y1="50.8" x2="48.26" y2="50.8" width="0" layer="19" extent="1-16"/>
 </signal>
 <signal name="N$37">
@@
 <contactref element="SW1" pad="2"/>
 <contactref element="R7" pad="2"/>
-<wire x1="48.26" y1="55.88" x2="48.26" y2="58.42" width="0" layer="19" extent="1-1"/>
-<wire x1="15.24" y1="55.88" x2="48.26" y2="55.88" width="0" layer="19" extent="1-1"/>
+<wire x1="15.24" y1="55.88" x2="48.26" y2="55.88" width="0.8128" layer="16"/>
+<wire x1="48.26" y1="58.42" x2="48.26" y2="55.88" width="0.8128" layer="16"/>
 </signal>
 <signal name="N$39">
 <contactref element="R8" pad="1"/>
 <contactref element="D1" pad="A"/>
-<wire x1="33.02" y1="50.8" x2="35.56" y2="50.8" width="0" layer="19" extent="1-1"/>
+<wire x1="35.56" y1="50.8" x2="33.02" y2="50.8" width="0.8128" layer="16"/>
 </signal>
 <signal name="N$40">
 <contactref element="D2" pad="A"/>
 <contactref element="R9" pad="1"/>
-<wire x1="27.94" y1="48.26" x2="35.56" y2="48.26" width="0" layer="19" extent="1-1"/>
+<wire x1="27.94" y1="48.26" x2="35.56" y2="48.26" width="0.8128" layer="16"/>
 </signal>
 </signals>
