File: eagle/OpenProg-18F2550-new.sch (EAGLE design)
At the start: 52 parts, among them J1 CONN-10P, J2 ICSP-IN, J3 USB-SH, J4 ICSP-OUT, T1 BC557, T2 BC557, T3 BC547, T4 BC547, U1 PIC18F2550-I/SP-V, X1 12MHz

Commit message: ...
Parts:
- added IC1: (no value), ic-package:DIL40
- R7: device r:R-H0204/10 -> r:R-H0204/10-V
- S1: value PUSHBUTTON-P1T -> PUSHBUTTONPB-2P1T; device sw:PUSHBUTTON-P1T -> sw:PUSHBUTTONPB-2P1T
Changed lines of the file:
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@@
 <part name="R8" library="r" deviceset="R-H" device="0204/10" value="2.2kΩ"/>
 <part name="S9" library="pad" deviceset="GND" device=""/>
-<part name="R7" library="r" deviceset="R-H" device="0204/10" value="1MΩ"/>
-<part name="S1" library="sw" deviceset="PUSHBUTTON" device="-P1T" value=""/>
+<part name="R7" library="r" deviceset="R-H" device="0204/10-V" value="1MΩ"/>
+<part name="S1" library="sw" deviceset="PUSHBUTTON" device="PB-2P1T" value="PUSHBUTTONPB-2P1T"/>
 <part name="D1" library="d" deviceset="LED" device="-3MM" value="YELLOW"/>
 <part name="D2" library="d" deviceset="LED" device="-3MM" value="GREEN"/>
@@
 <part name="DI" library="pad" deviceset="HPORT" device=""/>
 <part name="CKI" library="pad" deviceset="HPORT" device=""/>
+<part name="IC1" library="ic-package" deviceset="DIL40" device=""/>
 </parts>
 <sheets>
@@
 <instance part="DI" gate="1" x="132.08" y="35.56"/>
 <instance part="CKI" gate="1" x="132.08" y="33.02"/>
+<instance part="IC1" gate="G$1" x="257.81" y="35.56"/>
 </instances>
 <busses>
