File: eagle/OpenProg-18F2550-etch-it.brd (EAGLE design)
At the start: 52 parts, among them J1 CONN-10P, J2 ICSP-IN, J3 USB-SH, J4 ICSP-OUT, T1 BC557, T2 BC557, T3 BC547, T4 BC547, U1 PIC18F2550-I/SP-V, X1 12MHz

Commit message: ...
Parts:
- removed CKI, DI: HPORT, pad:SPAD
- removed J4: ICSP-OUT, pinconn:PIC-PK3
- moved C4 5.08 mm to (30.5, 12.7)
- moved R2 2.54 mm to (15.2, 53.3)
- moved R1 2.54 mm to (15.2, 55.9)
Connections:
- removed net N$2: CKI.1, J4.5
- removed net N$7: DI.1, J4.4
- net GND: no longer J4.3
- net VDDU: no longer J4.2
- net VPPU: no longer J4.1
Routing:
- net VCC: track 175.3 -> 212.6 mm
- net GND: track 213.6 -> 183.9 mm
- net VPPU: track 25.7 -> 7.90 mm, vias 2 -> 1
- net VDDU: track 22.9 -> 12.7 mm
- net N$36: track 2.54 -> 6.13 mm
- net N$7: track 2.54 -> 0.00 mm
- net N$2: track 2.54 -> 0.00 mm
- net VPP: track 34.8 -> 37.2 mm
- net N$34: track 15.2 -> 13.0 mm
- net FB: track 25.7 -> 27.9 mm
- net N$15: track 17.3 -> 16.2 mm
- net N$33: track 10.8 -> 9.72 mm
- net VPPCTL: track 7.62 -> 6.88 mm
- net N$1: track 10.2 -> 9.42 mm
- net OSC1: track 11.7 -> 11.2 mm
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
Commit message: ...
Parts:
- C7: device c:C025-015X024 -> c:C050-020X036
- moved C7 2.84 mm to (17.8, 12.7)
- moved ICSPVDD 2.54 mm to (10.2, 12.7)
- moved C4 2.54 mm to (30.5, 10.2)
- moved R25 2.54 mm to (15.2, 10.2)
- moved C2 1.80 mm to (26.7, 30.5), turned to 0 degrees
- moved C3 1.27 mm to (26.7, 26.7), turned to 0 degrees
Routing:
- net VCC: track 212.6 -> 214.7 mm
- net N$36: track 6.13 -> 8.22 mm
- net GND: track 183.9 -> 182.1 mm
- net VDDU: track 12.7 -> 13.8 mm
- net OSC2: track 11.2 -> 10.7 mm

Commit message: ...
Routing:
- net N$17: track 7.57 -> 2.54 mm
- net N$31: track 7.54 -> 2.51 mm
- net N$16: track 7.54 -> 2.51 mm
- net N$18: track 7.60 -> 2.66 mm
- net N$19: track 7.62 -> 2.70 mm
- net N$20: track 7.65 -> 2.75 mm
- net N$21: track 7.68 -> 2.80 mm
- net GND: track 182.1 -> 179.6 mm
- net VPPU: track 7.90 -> 5.36 mm
- added copper zone on layer 16, net GND

Commit message: ...
Parts:
- moved X1 1.27 mm to (31.8, 27.9)
Routing:
- net N$15: track 16.2 -> 14.6 mm
- net FB: track 27.9 -> 26.8 mm
- net N$1: track 9.42 -> 8.67 mm
- net OSC1: track 11.2 -> 10.7 mm
- added copper zone on layer 16, net N$2
- removed copper zone on layer 16, net GND

Commit message: ...
Parts:
- moved C3 1.27 mm to (26.7, 25.4)
- moved L1 1.27 mm to (10.2, 34.3)
Routing:
- net VCC: track 214.3 -> 218.7 mm
- net GND: track 179.5 -> 177.8 mm
- net N$5: track 5.08 -> 6.35 mm
- net VPPCTL: track 6.88 -> 6.13 mm
- removed copper zone on layer 16, net N$2
Other:
- board outline added: 68.6 x 61 mm
