File: eagle/broken/JDM2-2voltage-new.brd (EAGLE design)
At the start: 35.6 x 27.9 mm, 18 parts, among them J1 COMPORT-6PIN, J2 PIC-ICSPICSP, SW1 SL-SW-2P-2T-S, T1 BC547, T2 BC547

Commit message: ...
Changed lines of the file:
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@@
 <contactref element="J1" pad="5"/>
 <contactref element="R2" pad="1"/>
-<wire x1="1.27" y1="6.35" x2="3.81" y2="6.35" width="0.6096" layer="16"/>
-<wire x1="3.81" y1="6.35" x2="6.35" y2="6.35" width="0.6096" layer="16"/>
+<wire x1="1.27" y1="6.35" x2="3.81" y2="6.35" width="1.27" layer="16"/>
+<wire x1="3.81" y1="6.35" x2="6.35" y2="6.35" width="1.27" layer="16"/>
 </signal>
 <signal name="/MCLR">
@@
 <contactref element="D2" pad="A"/>
 <via x="13.97" y="8.89" extent="1-16" drill="0.6" shape="square"/>
-<wire x1="34.29" y1="8.89" x2="31.75" y2="8.89" width="0.6096" layer="16"/>
-<wire x1="31.75" y1="8.89" x2="13.97" y2="8.89" width="0.6096" layer="16"/>
-<wire x1="13.97" y1="8.89" x2="13.97" y2="19.05" width="0.6096" layer="1"/>
+<wire x1="34.29" y1="8.89" x2="31.75" y2="8.89" width="1.27" layer="16"/>
+<wire x1="31.75" y1="8.89" x2="13.97" y2="8.89" width="1.27" layer="16"/>
+<wire x1="13.97" y1="8.89" x2="13.97" y2="19.05" width="1.27" layer="1"/>
 <via x="13.97" y="19.05" extent="1-16" drill="0.6" shape="square"/>
 <wire x1="13.97" y1="19.05" x2="16.51" y2="19.05" width="0" layer="19" extent="1-1"/>
@@
 <contactref element="R3" pad="1"/>
 <contactref element="J2" pad="5"/>
-<wire x1="34.29" y1="1.27" x2="34.29" y2="3.81" width="0.6096" layer="16"/>
-<wire x1="16.51" y1="1.27" x2="34.29" y2="1.27" width="0.6096" layer="16"/>
+<wire x1="34.29" y1="1.27" x2="34.29" y2="3.81" width="1.27" layer="16"/>
+<wire x1="16.51" y1="1.27" x2="34.29" y2="1.27" width="1.27" layer="16"/>
 </signal>
 <signal name="TXD">
@@
 <contactref element="T1" pad="B"/>
 <contactref element="J1" pad="1"/>
-<wire x1="31.75" y1="16.51" x2="19.05" y2="16.51" width="0.6096" layer="16"/>
-<wire x1="1.27" y1="16.51" x2="10.16" y2="16.51" width="0.6096" layer="16"/>
-<wire x1="10.16" y1="16.51" x2="19.05" y2="16.51" width="0.6096" layer="16"/>
-<wire x1="19.05" y1="16.51" x2="19.05" y2="19.05" width="0.6096" layer="16"/>
-<wire x1="8.89" y1="19.05" x2="10.16" y2="16.51" width="0.6096" layer="16"/>
+<wire x1="31.75" y1="16.51" x2="19.05" y2="16.51" width="1.27" layer="16"/>
+<wire x1="1.27" y1="16.51" x2="10.16" y2="16.51" width="1.27" layer="16"/>
+<wire x1="10.16" y1="16.51" x2="19.05" y2="16.51" width="1.27" layer="16"/>
+<wire x1="19.05" y1="16.51" x2="19.05" y2="19.05" width="1.27" layer="16"/>
+<wire x1="8.89" y1="19.05" x2="10.16" y2="16.51" width="1.27" layer="16"/>
 </signal>
 <signal name="VPP">
@@
 <contactref element="R1" pad="1"/>
 <contactref element="T2" pad="B"/>
-<wire x1="8.89" y1="3.81" x2="6.35" y2="3.81" width="0.6096" layer="16"/>
+<wire x1="8.89" y1="3.81" x2="6.35" y2="3.81" width="1.27" layer="16"/>
 </signal>
 <signal name="DATA">
@@
 <via x="6.35" y="1.27" extent="1-16" drill="0.6"/>
 <via x="6.35" y="1.27" extent="1-16" drill="0.6"/>
-<wire x1="6.35" y1="1.27" x2="8.89" y2="1.27" width="0.6096" layer="16"/>
+<wire x1="6.35" y1="1.27" x2="8.89" y2="1.27" width="1.27" layer="16"/>
 </signal>
 <signal name="CLK">
@@
 <contactref element="J2" pad="4"/>
 <contactref element="J1" pad="4"/>
-<wire x1="11.43" y1="8.89" x2="11.43" y2="3.81" width="0.6096" layer="16"/>
-<wire x1="34.29" y1="6.35" x2="31.75" y2="6.35" width="0.6096" layer="16"/>
-<wire x1="31.75" y1="6.35" x2="31.75" y2="3.81" width="0.6096" layer="16"/>
-<wire x1="31.75" y1="3.81" x2="11.43" y2="3.81" width="0.6096" layer="16"/>
-<wire x1="6.35" y1="8.89" x2="1.27" y2="8.89" width="0.6096" layer="16"/>
-<wire x1="1.27" y1="8.89" x2="11.43" y2="8.89" width="0.6096" layer="16"/>
+<wire x1="11.43" y1="8.89" x2="11.43" y2="3.81" width="1.27" layer="16"/>
+<wire x1="34.29" y1="6.35" x2="31.75" y2="6.35" width="1.27" layer="16"/>
+<wire x1="31.75" y1="6.35" x2="31.75" y2="3.81" width="1.27" layer="16"/>
+<wire x1="31.75" y1="3.81" x2="11.43" y2="3.81" width="1.27" layer="16"/>
+<wire x1="6.35" y1="8.89" x2="1.27" y2="8.89" width="1.27" layer="16"/>
+<wire x1="1.27" y1="8.89" x2="11.43" y2="8.89" width="1.27" layer="16"/>
 </signal>
 <signal name="N$7">
 <contactref element="J1" pad="2"/>
 <contactref element="R2" pad="2"/>
-<wire x1="3.81" y1="13.97" x2="1.27" y2="13.97" width="0.6096" layer="16"/>
+<wire x1="3.81" y1="13.97" x2="1.27" y2="13.97" width="1.27" layer="16"/>
 </signal>
 <signal name="VCC">
@@
 <contactref element="R1" pad="2"/>
 <contactref element="J2" pad="2"/>
-<wire x1="26.67" y1="11.43" x2="34.29" y2="11.43" width="0.6096" layer="16"/>
-<wire x1="26.67" y1="11.43" x2="26.67" y2="21.59" width="0.6096" layer="1"/>
-<wire x1="26.67" y1="21.59" x2="26.67" y2="24.13" width="0.6096" layer="16"/>
+<wire x1="26.67" y1="11.43" x2="34.29" y2="11.43" width="1.27" layer="16"/>
+<wire x1="26.67" y1="11.43" x2="26.67" y2="21.59" width="1.27" layer="1"/>
+<wire x1="26.67" y1="21.59" x2="26.67" y2="24.13" width="1.27" layer="16"/>
 <via x="26.67" y="11.43" extent="1-16" drill="0.6" shape="square"/>
 <via x="26.67" y="21.59" extent="1-16" drill="0.6" shape="square"/>
-<wire x1="11.43" y1="11.43" x2="8.89" y2="11.43" width="0.6096" layer="16"/>
-<wire x1="1.27" y1="11.43" x2="8.89" y2="11.43" width="0.6096" layer="16"/>
+<wire x1="11.43" y1="11.43" x2="8.89" y2="11.43" width="1.27" layer="16"/>
+<wire x1="1.27" y1="11.43" x2="8.89" y2="11.43" width="1.27" layer="16"/>
 <contactref element="SW1" pad="5"/>
-<wire x1="26.67" y1="11.43" x2="16.51" y2="11.43" width="0.6096" layer="16"/>
-<wire x1="11.43" y1="11.43" x2="16.51" y2="11.43" width="0.6096" layer="16"/>
+<wire x1="26.67" y1="11.43" x2="16.51" y2="11.43" width="1.27" layer="16"/>
+<wire x1="11.43" y1="11.43" x2="16.51" y2="11.43" width="1.27" layer="16"/>
 <contactref element="D4A" pad="A"/>
 <contactref element="D4B" pad="A"/>
-<wire x1="8.89" y1="26.67" x2="8.89" y2="24.13" width="0.6096" layer="16"/>
-<wire x1="8.89" y1="24.13" x2="5.08" y2="21.59" width="0.6096" layer="16"/>
+<wire x1="8.89" y1="26.67" x2="8.89" y2="24.13" width="1.27" layer="16"/>
+<wire x1="8.89" y1="24.13" x2="5.08" y2="21.59" width="1.27" layer="16"/>
 <wire x1="8.89" y1="11.43" x2="5.08" y2="21.59" width="0" layer="19" extent="16-16"/>
 </signal>
@@
 <contactref element="D5B" pad="A"/>
 <contactref element="D5A" pad="A"/>
-<wire x1="34.29" y1="13.97" x2="29.21" y2="13.97" width="0.6096" layer="16"/>
-<wire x1="29.21" y1="13.97" x2="24.13" y2="13.97" width="0.6096" layer="16"/>
-<wire x1="24.13" y1="13.97" x2="16.51" y2="13.97" width="0.6096" layer="16"/>
-<wire x1="16.51" y1="13.97" x2="6.35" y2="13.97" width="0.6096" layer="16"/>
+<wire x1="34.29" y1="13.97" x2="29.21" y2="13.97" width="1.27" layer="16"/>
+<wire x1="29.21" y1="13.97" x2="24.13" y2="13.97" width="1.27" layer="16"/>
+<wire x1="24.13" y1="13.97" x2="16.51" y2="13.97" width="1.27" layer="16"/>
+<wire x1="16.51" y1="13.97" x2="6.35" y2="13.97" width="1.27" layer="16"/>
 <wire x1="6.35" y1="13.97" x2="12.7" y2="19.05" width="0" layer="19" extent="1-1"/>
 <wire x1="8.89" y1="13.97" x2="6.35" y2="13.97" width="0" layer="19" extent="1-1"/>
@@
 <contactref element="C1" pad="+"/>
 <contactref element="SW1" pad="2"/>
-<wire x1="26.67" y1="26.67" x2="25.4" y2="25.4" width="0.6096" layer="16"/>
-<wire x1="25.4" y1="25.4" x2="19.05" y2="25.4" width="0.6096" layer="16"/>
-<wire x1="19.05" y1="25.4" x2="19.05" y2="24.13" width="0.6096" layer="16"/>
+<wire x1="26.67" y1="26.67" x2="25.4" y2="25.4" width="1.27" layer="16"/>
+<wire x1="25.4" y1="25.4" x2="19.05" y2="25.4" width="1.27" layer="16"/>
+<wire x1="19.05" y1="25.4" x2="19.05" y2="24.13" width="1.27" layer="16"/>
 <wire x1="21.59" y1="19.05" x2="19.05" y2="24.13" width="0" layer="19" extent="16-16"/>
 <wire x1="12.7" y1="21.59" x2="19.05" y2="25.4" width="0" layer="19" extent="16-16"/>
@@
 <contactref element="D4B" pad="C"/>
 <contactref element="SW1" pad="3"/>
-<wire x1="24.13" y1="26.67" x2="13.97" y2="26.67" width="0.6096" layer="16"/>
+<wire x1="24.13" y1="26.67" x2="13.97" y2="26.67" width="1.27" layer="16"/>
 </signal>
 <signal name="N$3">
 <contactref element="SW1" pad="4"/>
 <contactref element="D5A" pad="C"/>
-<wire x1="29.21" y1="21.59" x2="29.21" y2="24.13" width="0.6096" layer="16"/>
+<wire x1="29.21" y1="21.59" x2="29.21" y2="24.13" width="1.27" layer="16"/>
 </signal>
 <signal name="N$6">
 <contactref element="SW1" pad="6"/>
 <contactref element="D5B" pad="C"/>
-<wire x1="24.13" y1="21.59" x2="24.13" y2="24.13" width="0.6096" layer="16"/>
+<wire x1="24.13" y1="21.59" x2="24.13" y2="24.13" width="1.27" layer="16"/>
 </signal>
 </signals>
